File: ihc_mon.brd (EAGLE design)
At the start: 54.6 x 70.8 mm, 24 parts, among them IC1 PIC18F1220P, IC2 OX-52 10mhz, IC3 LX2885IGW, X1 22-23-2021

Commit message: uploads
Parts:
- added X2: 22-23-2021, con-molex:22-23-2021
- moved JP1 6.48 mm to (19.1, 72.4)
- moved R7 3.81 mm to (19.1, 25.4)
- moved C4 2.54 mm to (10.2, 26.7)
- moved C1 1.27 mm to (6.35, 33.0)
- moved C2 1.27 mm to (6.35, 49.5)
- moved D2 1.27 mm to (10.2, 20.3)
- moved R5 1.27 mm to (6.35, 43.2)
- moved R6 1.27 mm to (6.35, 38.1)
Connections:
- new net N$10: IC1.17, X2.1
- net VSS: now also D1.5, D1.8, D2.5, D2.8, X2.2
Routing:
- net VSS: track 120.8 -> 175.9 mm
- net N$10: track 0.00 -> 32.8 mm
- net VDD: track 148.3 -> 130.0 mm
- net N$20: track 70.6 -> 77.8 mm
- net N$15: track 51.7 -> 55.6 mm
- net N$12: track 33.5 -> 36.6 mm
- net N$21: track 66.6 -> 69.3 mm
- net N$7: track 12.3 -> 14.6 mm
- net N$5: track 5.58 -> 4.35 mm
Other:
- board size 54.6 x 70.8 mm -> 55.9 x 70.8 mm

Commit message: updates
Parts:
- added C8: 22, resistor:C025-024X044
- moved IC3 2.84 mm to (29.2, 43.2)
- moved R1 2.84 mm to (20.3, 49.5), turned to 90 degrees
- moved R9 2.84 mm to (20.3, 36.8), turned to 90 degrees
- moved R2 2.54 mm to (20.3, 43.2), turned to 90 degrees
- moved C3 1.27 mm to (19.1, 61.0)
- moved C5 1.27 mm to (22.9, 61.0)
Connections:
- net VDD: now also C8.1
- net VSS: now also C8.2
Routing:
- net N$21: track 69.3 -> 54.1 mm
- net VDD: track 130.0 -> 141.7 mm
- net N$24: track 27.9 -> 20.5 mm
- net N$15: track 55.6 -> 52.4 mm
- net N$23: track 19.9 -> 16.8 mm
- net N$4: track 3.82 -> 6.87 mm
- net N$26: track 3.96 -> 6.91 mm
- net N$3: track 4.05 -> 6.95 mm
- net N$10: track 32.8 -> 35.6 mm
- net N$20: track 77.8 -> 75.1 mm
- net N$11: track 27.7 -> 25.3 mm
- net N$22: track 27.2 -> 25.2 mm
- net N$19: track 22.3 -> 24.2 mm
- net N$18: track 13.6 -> 11.7 mm
- net N$9: track 3.91 -> 5.77 mm
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
Commit message: up
Parts:
- removed C8: 22, resistor:C025-024X044
- removed D1: HFBR1528, opto-transmittter-hp:HFBR25XX
- removed D2: HFBR2528, opto-transmittter-hp:HFBR25XX
- removed IC3: LX2885IGW, ic-package:SOCKET-16
- removed R10, R3, R4, R5, R9: 510, resistor:0204V
- removed R6: 10000, resistor:0204V
- removed R7: 2200, resistor:0204V
- removed R8: 100, resistor:0204V
- added C9: 0.1, rcl:C0805
- C1, C7: value 22 -> 22uf; device resistor:C025-024X044 -> rcl:C0805
- C2, C3, C4, C5: device resistor:C050-025X075 -> rcl:C0805
- C6: value 0.1 -> 22uf; device resistor:C050-025X075 -> rcl:C0805
- R1: value 510 -> 300; device resistor:0204V -> rcl:R0805
- R2: value 510 -> 10000; device resistor:0204V -> rcl:R0805
- moved C7 35.9 mm to (20.3, 59.7)
- moved X1 32.1 mm to (11.4, 17.8), turned to 0 degrees
- moved C1 22.9 mm to (27.9, 40.6), turned to 0 degrees
- moved C5 20.3 mm to (22.9, 40.6), turned to 0 degrees
- moved R1 16.5 mm to (5.08, 43.2), turned to 0 degrees
- moved R2 16.1 mm to (5.08, 38.1), turned to 180 degrees
- moved X2 13.1 mm to (30.5, 63.5)
- moved C6 10.9 mm to (16.5, 25.4), turned to 180 degrees
- moved C3 4.02 mm to (20.3, 64.8), turned to 0 degrees
- moved JP1 2.84 mm to (20.3, 74.9)
- moved IC2 2.84 mm to (10.2, 62.2)
- moved C2 1.80 mm to (5.08, 48.3), turned to 0 degrees
- moved C4 1.80 mm to (11.4, 25.4)
Connections:
- removed net N$1: IC3.1, R1.2
- removed net N$11: IC1.8, IC3.10
- removed net N$14: D1.2, IC1.9
- removed net N$16: IC1.1, R1.1
- removed net N$17: IC1.2, IC3.2
- removed net N$18: IC1.6, R2.1
- removed net N$19: IC1.7, IC3.3
- removed net N$2: IC3.4, R2.2
- removed net N$22: IC1.15, R4.2
- removed net N$23: IC1.18, IC3.14
- removed net N$24: IC1.3, IC3.8
- removed net N$26: IC3.9, R10.1
- removed net N$3: IC3.16, R3.1
- removed net N$4: IC3.13, R4.1
- removed net N$7: D2.1, IC1.10, R7.2
- removed net N$8: D1.1, R8.1
- removed net N$9: IC3.7, R9.2
- net N$12: now also R1.1, R2.2; no longer R5.1, R6.2
- net N$20: no longer R3.2
- net N$21: no longer IC3.15
- net N$5: now also R1.2; no longer R5.2
- net VDD: now also C9.2, R2.1; no longer C8.1, D2.3, R10.2, R6.1, R7.1, R8.2, R9.1
- net VSS: now also C9.1; no longer C8.2, D1.5, D1.8, D2.2, D2.5, D2.8
Routing:
- net VSS: track 177.4 -> 58.3 mm, vias 0 -> 1
- net N$20: track 75.1 -> 49.6 mm, vias 0 -> 1
- net N$11: track 25.3 -> 0.00 mm
- net N$22: track 25.2 -> 0.00 mm
- net N$14: track 24.5 -> 0.00 mm
- net N$19: track 24.2 -> 0.00 mm
- net N$24: track 20.5 -> 0.00 mm
- net VDD: track 141.7 -> 123.0 mm, vias 0 -> 1
- net N$17: track 17.2 -> 0.00 mm
- net N$23: track 16.8 -> 0.00 mm
- net N$10: track 35.6 -> 20.0 mm
- net N$7: track 14.6 -> 0.00 mm
- net N$18: track 11.7 -> 0.00 mm
- net N$16: track 11.2 -> 0.00 mm
- net N$8: track 9.71 -> 0.00 mm
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- added copper zone on layer 16, net VSS

Commit message: up
Parts:
- added ANALOG_OUT: CC MODE SIGNAL, con-molex:22-23-2021
- added C10: 0.1, rcl:C0805
- added C11, C8: 22uf, rcl:C0805
- added IC3: ADM3095EBRZ, SamacSys_Parts:SOIC127P600X175-16N
- added JP2: RS485, pinhead:1X06
- added L1: 10uh, rcl:0204/7
- added LED1: DATA, led:CHIPLED_0805
- added R3: 300, rcl:R0805
- added R4: 10000, rcl:R0805
- added R5: 2.2k, rcl:R0805
Connections:
- new net N$1: IC1.10, IC3.7
- new net N$11: ANALOG_OUT.1, C11.1, L1.2, R4.1
- new net N$13: LED1.A, R5.1
- new net N$14: IC1.3, R5.2
- new net N$2: IC1.9, IC3.4
- new net N$3: IC1.1, IC3.5
- new net N$4: IC1.2, IC3.6
- new net N$6: IC1.18, R3.1
- new net N$7: L1.1, R3.2
- new net N$8: IC3.14, JP2.2
- new net N$9: IC3.11, JP2.3
- net VDD: now also C10.1, C8.1, IC3.2, IC3.3, JP2.1
- net VSS: now also ANALOG_OUT.2, C10.2, C11.2, C8.2, IC3.1, IC3.10, IC3.12, IC3.13, IC3.15, IC3.16, IC3.8, IC3.9, JP2.4, LED1.C, R4.2
Routing:
- net VDD: track 123.0 -> 234.5 mm
- net VSS: track 58.3 -> 122.8 mm, vias 1 -> 3
- net N$14: track 0.00 -> 43.9 mm
- net N$4: track 0.00 -> 38.1 mm, vias 0 -> 1
- net N$3: track 0.00 -> 33.3 mm, vias 0 -> 1
- net N$2: track 0.00 -> 26.6 mm
- net N$11: track 0.00 -> 26.4 mm
- net N$1: track 0.00 -> 17.9 mm
- net N$13: track 0.00 -> 14.4 mm
- net N$6: track 0.00 -> 13.4 mm
- net N$15: track 58.7 -> 48.0 mm, vias 0 -> 1
- net N$7: track 0.00 -> 9.53 mm
- net N$9: track 0.00 -> 9.41 mm
- net N$8: track 0.00 -> 8.76 mm
- net N$20: track 49.6 -> 47.6 mm, vias 1 -> 0
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- added copper zone on layer 1, net VSS
Other:
- board text added: "RE20A RS485 FGB 1.0"

Commit message: up
Parts:
- added JP3: SIG, pinhead:1X06
- added LSP1: SE14, solpad:SE14
- added PAD1: (no value), wirepad:3,81/1,4
- added PAD2: (no value), wirepad:SMD1,27-2,54
- added R6: 10000, rcl:R0805
- added R8: 120, rcl:M1206
Connections:
- new net N$17: IC1.8, JP3.2
- new net N$18: IC1.6, JP3.3
- new net N$19: IC1.7, JP3.4
- new net N$22: IC1.15, JP3.5
- net N$1: now also R6.1
- net N$8: now also R8.1
- net N$9: now also R8.2
- net VDD: now also JP3.6, R6.2
- net VSS: now also JP2.5, JP2.6, JP3.1, LSP1.MP, PAD1.1, PAD2.1
Routing:
- net N$3: track 33.3 -> 72.3 mm, vias 1 -> 0
- net VDD: track 234.5 -> 195.8 mm, vias 1 -> 3
- net N$22: track 0.00 -> 28.4 mm, vias 0 -> 1
- net VSS: track 122.8 -> 147.9 mm
- net N$19: track 0.00 -> 17.2 mm
- net N$9: track 9.41 -> 23.5 mm
- net N$18: track 0.00 -> 14.0 mm
- net N$8: track 8.76 -> 20.0 mm
- net N$14: track 43.9 -> 34.7 mm, vias 0 -> 1
- net N$1: track 17.9 -> 26.5 mm, vias 0 -> 1
- net N$15: track 48.0 -> 55.6 mm
- net N$17: track 0.00 -> 6.65 mm
- net N$20: track 47.6 -> 42.3 mm
- net N$21: track 44.4 -> 41.4 mm, vias 2 -> 1
- net N$4: track 38.1 -> 39.9 mm, vias 1 -> 0
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Other:
- board text added: "RE20A RS485 FGB 1.1"
- board text removed: "RE20A RS485 FGB 1.0"

Commit message: up
Parts:
- added A4: a4, wirepad:SMD1,27-2,54
- C11: value 22uf -> 3.3uf
- GND1, GND2: value (none) -> gnd
- R3: value 300 -> 100
- R4: value 10000 -> 2200
- R5: value 2.2k -> 1000
- renumbered PAD1 to GND1, PAD2 to GND2
Connections:
- removed net N$14: IC1.3, R5.2
- new net N$16: A4.1, IC1.3
- net N$17: now also R5.2
Routing:
- net N$3: track 72.3 -> 33.3 mm, vias 0 -> 1
- net N$14: track 34.7 -> 0.00 mm, vias 1 -> 0
- net N$20: track 42.3 -> 75.7 mm
- net N$17: track 6.65 -> 35.0 mm
- net N$16: track 0.00 -> 18.8 mm
- net VDD: track 195.8 -> 212.7 mm
- net VSS: track 147.9 -> 157.5 mm, vias 3 -> 1
- net N$21: track 41.4 -> 49.3 mm, vias 1 -> 0
- net N$15: track 55.6 -> 48.0 mm
- net N$4: track 39.9 -> 46.7 mm
- net N$1: track 26.5 -> 20.0 mm, vias 1 -> 0
- net N$10: track 22.8 -> 26.0 mm
- net N$22: track 28.4 -> 30.9 mm, vias 1 -> 0
- net N$2: track 26.9 -> 28.7 mm
- net N$19: track 17.2 -> 16.4 mm

Commit message: up
Parts:
- removed IC2: OX-52 10mhz, ic-package:SOCKET-08
- removed L1: 10uh, rcl:0204/7
- added L2: 100uh, inductor-neosid:SM-1206
- added LED2: DATA, led:CHIPLED_1206
- added OS1: 10MHz, IQD-Frequency-Products:7.2X5.2-4-PAD
- added R7: 1000, rcl:R0805
- added R9: 300, rcl:R0805
- LED1: value DATA -> POWER; device led:CHIPLED_0805 -> led:CHIPLED_1206
- moved LED1 57.5 mm to (8.89, 71.1)
Connections:
- new net N$14: LED1.A, R7.1
- new net N$23: C2.1, R1.1, R2.2, R9.2
- net N$11: now also L2.2; no longer L1.2
- net N$12: now also R9.1; no longer C2.1, R1.1, R2.2
- net N$13: now also LED2.A; no longer LED1.A
- net N$25: now also OS1.3; no longer IC2.5
- net N$7: now also L2.1; no longer L1.1
- net VDD: now also OS1.1, OS1.4, R7.2; no longer IC2.1, IC2.8
- net VSS: now also LED2.C, OS1.2; no longer IC2.4
Routing:
- net VDD: track 212.7 -> 284.7 mm, vias 3 -> 1
- net VSS: track 157.5 -> 176.3 mm
- net N$20: track 75.7 -> 57.0 mm, vias 0 -> 1
- net N$23: track 0.00 -> 16.0 mm
- net N$12: track 40.9 -> 29.0 mm
- net N$4: track 46.7 -> 37.0 mm, vias 0 -> 1
- net N$25: track 14.4 -> 21.8 mm, vias 0 -> 1
- net N$14: track 0.00 -> 3.77 mm
- net N$21: track 49.3 -> 52.4 mm
- net N$19: track 16.4 -> 14.0 mm
- net N$11: track 26.4 -> 24.2 mm
- net N$17: track 35.0 -> 32.9 mm
- net N$18: track 14.0 -> 15.7 mm
- net N$2: track 28.7 -> 30.3 mm
- net N$15: track 48.0 -> 49.4 mm, vias 1 -> 0
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
Commit message: up
Parts:
- R5, R7: value 1000 -> 1.47k
Changed lines of the file:
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@@
 <attribute name="VALUE" x="46.355" y="64.77" size="1.27" layer="27" rot="R180"/>
 </element>
-<element name="R5" library="rcl" library_urn="urn:adsk.eagle:library:334" package="R0805" package3d_urn="urn:adsk.eagle:package:23553/2" value="1000" x="26.67" y="21.59" smashed="yes">
+<element name="R5" library="rcl" library_urn="urn:adsk.eagle:library:334" package="R0805" package3d_urn="urn:adsk.eagle:package:23553/2" value="1.47k" x="26.67" y="21.59" smashed="yes">
 <attribute name="NAME" x="26.035" y="22.86" size="1.27" layer="25"/>
 <attribute name="POPULARITY" value="85" x="26.67" y="21.59" size="1.778" layer="27" display="off"/>
@@
 <attribute name="VALUE" x="39.37" y="24.13" size="1.27" layer="27" rot="R180"/>
 </element>
-<element name="R7" library="rcl" library_urn="urn:adsk.eagle:library:334" package="R0805" package3d_urn="urn:adsk.eagle:package:23553/2" value="1000" x="15.24" y="71.12" smashed="yes">
+<element name="R7" library="rcl" library_urn="urn:adsk.eagle:library:334" package="R0805" package3d_urn="urn:adsk.eagle:package:23553/2" value="1.47k" x="15.24" y="71.12" smashed="yes">
 <attribute name="NAME" x="18.415" y="71.12" size="1.27" layer="25"/>
 <attribute name="POPULARITY" value="85" x="15.24" y="71.12" size="1.778" layer="27" display="off"/>
