File: ihc_mon.brd (EAGLE design)
At the start: 55.9 x 70.8 mm, 36 parts, among them IC1 PIC18F1220P, IC3 ADM3095EBRZ, X1 22-23-2021, X2 22-23-2021

Commit message: up
Parts:
- R1: value 300 -> 100
- R9: value 300 -> 50
Changed lines of the file:
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@@
 <attribute name="VALUE" x="19.05" y="57.15" size="1.27" layer="27"/>
 </element>
-<element name="R1" library="rcl" library_urn="urn:adsk.eagle:library:334" package="R0805" package3d_urn="urn:adsk.eagle:package:23553/2" value="300" x="5.08" y="43.18" smashed="yes">
+<element name="R1" library="rcl" library_urn="urn:adsk.eagle:library:334" package="R0805" package3d_urn="urn:adsk.eagle:package:23553/2" value="100" x="5.08" y="43.18" smashed="yes">
 <attribute name="NAME" x="4.445" y="44.45" size="1.27" layer="25"/>
 <attribute name="POPULARITY" value="85" x="5.08" y="43.18" size="1.778" layer="27" display="off"/>
@@
 <attribute name="VALUE" x="10.16" y="73.66" size="1.27" layer="27" rot="R180"/>
 </element>
-<element name="R9" library="rcl" library_urn="urn:adsk.eagle:library:334" package="R0805" package3d_urn="urn:adsk.eagle:package:23553/2" value="300" x="5.08" y="53.34" smashed="yes">
+<element name="R9" library="rcl" library_urn="urn:adsk.eagle:library:334" package="R0805" package3d_urn="urn:adsk.eagle:package:23553/2" value="50" x="5.08" y="53.34" smashed="yes">
 <attribute name="NAME" x="4.445" y="54.61" size="1.27" layer="25"/>
 <attribute name="POPULARITY" value="85" x="5.08" y="53.34" size="1.778" layer="27" display="off"/>

Commit message: up
Parts:
- R1: value 100 -> 50
- R9: value 50 -> 0
Changed lines of the file:
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@@
 <attribute name="VALUE" x="19.05" y="57.15" size="1.27" layer="27"/>
 </element>
-<element name="R1" library="rcl" library_urn="urn:adsk.eagle:library:334" package="R0805" package3d_urn="urn:adsk.eagle:package:23553/2" value="100" x="5.08" y="43.18" smashed="yes">
+<element name="R1" library="rcl" library_urn="urn:adsk.eagle:library:334" package="R0805" package3d_urn="urn:adsk.eagle:package:23553/2" value="50" x="5.08" y="43.18" smashed="yes">
 <attribute name="NAME" x="4.445" y="44.45" size="1.27" layer="25"/>
 <attribute name="POPULARITY" value="85" x="5.08" y="43.18" size="1.778" layer="27" display="off"/>
@@
 <attribute name="VALUE" x="10.16" y="73.66" size="1.27" layer="27" rot="R180"/>
 </element>
-<element name="R9" library="rcl" library_urn="urn:adsk.eagle:library:334" package="R0805" package3d_urn="urn:adsk.eagle:package:23553/2" value="50" x="5.08" y="53.34" smashed="yes">
+<element name="R9" library="rcl" library_urn="urn:adsk.eagle:library:334" package="R0805" package3d_urn="urn:adsk.eagle:package:23553/2" value="0" x="5.08" y="53.34" smashed="yes">
 <attribute name="NAME" x="4.445" y="54.61" size="1.27" layer="25"/>
 <attribute name="POPULARITY" value="85" x="5.08" y="53.34" size="1.778" layer="27" display="off"/>

Commit message: up
Parts:
- R5, R7: value 1.47k -> 2k
Changed lines of the file:
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@@
 <attribute name="VALUE" x="46.355" y="64.77" size="1.27" layer="27" rot="R180"/>
 </element>
-<element name="R5" library="rcl" library_urn="urn:adsk.eagle:library:334" package="R0805" package3d_urn="urn:adsk.eagle:package:23553/2" value="1.47k" x="26.67" y="21.59" smashed="yes">
+<element name="R5" library="rcl" library_urn="urn:adsk.eagle:library:334" package="R0805" package3d_urn="urn:adsk.eagle:package:23553/2" value="2k" x="26.67" y="21.59" smashed="yes">
 <attribute name="NAME" x="26.035" y="22.86" size="1.27" layer="25"/>
 <attribute name="POPULARITY" value="85" x="26.67" y="21.59" size="1.778" layer="27" display="off"/>
@@
 <attribute name="VALUE" x="39.37" y="24.13" size="1.27" layer="27" rot="R180"/>
 </element>
-<element name="R7" library="rcl" library_urn="urn:adsk.eagle:library:334" package="R0805" package3d_urn="urn:adsk.eagle:package:23553/2" value="1.47k" x="15.24" y="71.12" smashed="yes">
+<element name="R7" library="rcl" library_urn="urn:adsk.eagle:library:334" package="R0805" package3d_urn="urn:adsk.eagle:package:23553/2" value="2k" x="15.24" y="71.12" smashed="yes">
 <attribute name="NAME" x="18.415" y="71.12" size="1.27" layer="25"/>
 <attribute name="POPULARITY" value="85" x="15.24" y="71.12" size="1.778" layer="27" display="off"/>
