File: ihc_mon.sch (EAGLE design)
At the start: 24 parts, among them IC1 PIC18F1220P, IC2 OX-52 10mhz, IC3 LX2885IGW, X1 22-23-2021

Commit message: uploads
Parts:
- added X2: 22-23-2021, con-molex:22-23-2021
Connections:
- new net N$10: IC1.INT2/P1B/RB2, X2-1.S
- net VSS: now also D1.GND, D1.GND@1, D2.1, D2.4, X2-2.S
Changed lines of the file:
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@@
 <?xml version="1.0" encoding="utf-8"?>
 <!DOCTYPE eagle SYSTEM "eagle.dtd">
-<eagle version="7.6.0">
+<eagle version="7.7.0">
 <drawing>
 <settings>
@@
 <part name="VSS1" library="supply1" deviceset="VSS" device=""/>
 <part name="VSS2" library="supply1" deviceset="VSS" device=""/>
+<part name="X2" library="con-molex" deviceset="22-23-2021" device=""/>
+<part name="VSS3" library="supply1" deviceset="VSS" device=""/>
+<part name="VSS4" library="supply1" deviceset="VSS" device=""/>
 </parts>
 <sheets>
@@
 <instance part="VSS1" gate="G$1" x="99.06" y="-15.24"/>
 <instance part="VSS2" gate="G$1" x="-17.78" y="-17.78"/>
+<instance part="X2" gate="-1" x="119.38" y="27.94"/>
+<instance part="X2" gate="-2" x="119.38" y="25.4"/>
+<instance part="VSS3" gate="G$1" x="111.76" y="22.86"/>
+<instance part="VSS4" gate="G$1" x="45.72" y="-22.86"/>
 </instances>
 <busses>
@@
 <wire x1="15.24" y1="30.48" x2="17.78" y2="30.48" width="0.1524" layer="91"/>
 <junction x="17.78" y="30.48"/>
-</segment>
-</net>
-<net name="N$6" class="0">
-<segment>
-<pinref part="R5" gate="G$1" pin="1"/>
-<pinref part="R6" gate="G$1" pin="2"/>
-<pinref part="C2" gate="G$1" pin="1"/>
-<junction x="5.08" y="30.48"/>
-<pinref part="C2" gate="G$1" pin="1"/>
-<wire x1="5.08" y1="30.48" x2="7.62" y2="33.02" width="0.1524" layer="91"/>
-<wire x1="7.62" y1="33.02" x2="-12.7" y2="33.02" width="0.1524" layer="91"/>
-<wire x1="-12.7" y1="33.02" x2="-12.7" y2="17.78" width="0.1524" layer="91"/>
-<wire x1="-12.7" y1="17.78" x2="111.76" y2="17.78" width="0.1524" layer="91"/>
-<pinref part="JP1" gate="A" pin="1"/>
-<wire x1="111.76" y1="17.78" x2="111.76" y2="15.24" width="0.1524" layer="91"/>
-<junction x="5.08" y="30.48"/>
-<junction x="111.76" y="15.24"/>
 </segment>
 </net>
@@
 <junction x="-17.78" y="-15.24"/>
 </segment>
-</net>
+<segment>
+<pinref part="X2" gate="-2" pin="S"/>
+<wire x1="116.84" y1="25.4" x2="111.76" y2="25.4" width="0.1524" layer="91"/>
+<pinref part="VSS3" gate="G$1" pin="VSS"/>
+</segment>
+<segment>
+<pinref part="D2" gate="G$1" pin="4"/>
+<pinref part="D2" gate="G$1" pin="1"/>
+<wire x1="35.56" y1="-20.32" x2="35.56" y2="-22.86" width="0.1524" layer="91"/>
+<wire x1="35.56" y1="-20.32" x2="45.72" y2="-20.32" width="0.1524" layer="91"/>
+<wire x1="45.72" y1="-20.32" x2="45.72" y2="-15.24" width="0.1524" layer="91"/>
+<pinref part="D1" gate="G$1" pin="GND@1"/>
+<pinref part="D1" gate="G$1" pin="GND"/>
+<wire x1="53.34" y1="-15.24" x2="53.34" y2="-17.78" width="0.1524" layer="91"/>
+<wire x1="45.72" y1="-15.24" x2="53.34" y2="-15.24" width="0.1524" layer="91"/>
+<pinref part="VSS4" gate="G$1" pin="VSS"/>
+<junction x="45.72" y="-20.32"/>
+<junction x="53.34" y="-15.24"/>
+<junction x="35.56" y="-20.32"/>
+</segment>
+</net>
+<net name="N$10" class="0">
+<segment>
+<pinref part="IC1" gate="G$1" pin="INT2/P1B/RB2"/>
+<wire x1="76.2" y1="45.72" x2="114.3" y2="45.72" width="0.1524" layer="91"/>
+<wire x1="114.3" y1="45.72" x2="114.3" y2="27.94" width="0.1524" layer="91"/>
+<pinref part="X2" gate="-1" pin="S"/>
+<wire x1="114.3" y1="27.94" x2="116.84" y2="27.94" width="0.1524" layer="91"/>
+</segment>
+</net>
+<net name="N$12" class="0">
+<segment>
+<pinref part="R5" gate="G$1" pin="1"/>
+<pinref part="R6" gate="G$1" pin="2"/>
+<pinref part="C2" gate="G$1" pin="1"/>
+<junction x="5.08" y="30.48"/>
+<junction x="5.08" y="30.48"/>
+<wire x1="5.08" y1="30.48" x2="5.08" y2="33.02" width="0.1524" layer="91"/>
+<wire x1="-12.7" y1="33.02" x2="-12.7" y2="17.78" width="0.1524" layer="91"/>
+<wire x1="-12.7" y1="17.78" x2="111.76" y2="17.78" width="0.1524" layer="91"/>
+<pinref part="JP1" gate="A" pin="1"/>
+<wire x1="111.76" y1="17.78" x2="111.76" y2="15.24" width="0.1524" layer="91"/>
+<junction x="111.76" y="15.24"/>
+<wire x1="5.08" y1="33.02" x2="-12.7" y2="33.02" width="0.1524" layer="91"/>
+</segment>
+</net>

Commit message: updates
Parts:
- added C8: 22, resistor:C-US025-024X044
- IC1: MPN (none) -> PIC18F1320-I/P
Connections:
- net VDD: now also C8.1
- net VSS: now also C8.2
Changed lines of the file:
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@@
 <grid distance="0.1" unitdist="inch" unit="inch" style="lines" multiple="1" display="no" altdistance="0.01" altunitdist="inch" altunit="inch"/>
 <layers>
-<layer number="1" name="Top" color="4" fill="1" visible="no" active="no"/>
-<layer number="2" name="Route2" color="1" fill="3" visible="no" active="no"/>
-<layer number="3" name="Route3" color="4" fill="3" visible="no" active="no"/>
-<layer number="14" name="Route14" color="1" fill="6" visible="no" active="no"/>
-<layer number="15" name="Route15" color="4" fill="6" visible="no" active="no"/>
-<layer number="16" name="Bottom" color="1" fill="1" visible="no" active="no"/>
-<layer number="17" name="Pads" color="2" fill="1" visible="no" active="no"/>
-<layer number="18" name="Vias" color="2" fill="1" visible="no" active="no"/>
-<layer number="19" name="Unrouted" color="6" fill="1" visible="no" active="no"/>
-<layer number="20" name="Dimension" color="15" fill="1" visible="no" active="no"/>
-<layer number="21" name="tPlace" color="7" fill="1" visible="no" active="no"/>
-<layer number="22" name="bPlace" color="7" fill="1" visible="no" active="no"/>
-<layer number="23" name="tOrigins" color="15" fill="1" visible="no" active="no"/>
-<layer number="24" name="bOrigins" color="15" fill="1" visible="no" active="no"/>
-<layer number="25" name="tNames" color="7" fill="1" visible="no" active="no"/>
-<layer number="26" name="bNames" color="7" fill="1" visible="no" active="no"/>
-<layer number="27" name="tValues" color="7" fill="1" visible="no" active="no"/>
-<layer number="28" name="bValues" color="7" fill="1" visible="no" active="no"/>
+<layer number="1" name="Top" color="4" fill="1" visible="yes" active="no"/>
+<layer number="2" name="Route2" color="1" fill="3" visible="yes" active="no"/>
+<layer number="3" name="Route3" color="4" fill="3" visible="yes" active="no"/>
+<layer number="14" name="Route14" color="1" fill="6" visible="yes" active="no"/>
+<layer number="15" name="Route15" color="4" fill="6" visible="yes" active="no"/>
+<layer number="16" name="Bottom" color="1" fill="1" visible="yes" active="no"/>
+<layer number="17" name="Pads" color="2" fill="1" visible="yes" active="no"/>
+<layer number="18" name="Vias" color="2" fill="1" visible="yes" active="no"/>
+<layer number="19" name="Unrouted" color="6" fill="1" visible="yes" active="no"/>
+<layer number="20" name="Dimension" color="15" fill="1" visible="yes" active="no"/>
+<layer number="21" name="tPlace" color="7" fill="1" visible="yes" active="no"/>
+<layer number="22" name="bPlace" color="7" fill="1" visible="yes" active="no"/>
+<layer number="23" name="tOrigins" color="15" fill="1" visible="yes" active="no"/>
+<layer number="24" name="bOrigins" color="15" fill="1" visible="yes" active="no"/>
+<layer number="25" name="tNames" color="7" fill="1" visible="yes" active="no"/>
+<layer number="26" name="bNames" color="7" fill="1" visible="yes" active="no"/>
+<layer number="27" name="tValues" color="7" fill="1" visible="yes" active="no"/>
+<layer number="28" name="bValues" color="7" fill="1" visible="yes" active="no"/>
 <layer number="29" name="tStop" color="7" fill="3" visible="no" active="no"/>
 <layer number="30" name="bStop" color="7" fill="6" visible="no" active="no"/>
@@
 <layer number="35" name="tGlue" color="7" fill="4" visible="no" active="no"/>
 <layer number="36" name="bGlue" color="7" fill="5" visible="no" active="no"/>
-<layer number="37" name="tTest" color="7" fill="1" visible="no" active="no"/>
-<layer number="38" name="bTest" color="7" fill="1" visible="no" active="no"/>
+<layer number="37" name="tTest" color="7" fill="1" visible="yes" active="no"/>
+<layer number="38" name="bTest" color="7" fill="1" visible="yes" active="no"/>
 <layer number="39" name="tKeepout" color="4" fill="11" visible="no" active="no"/>
 <layer number="40" name="bKeepout" color="1" fill="11" visible="no" active="no"/>
@@
 <layer number="44" name="Drills" color="7" fill="1" visible="no" active="no"/>
 <layer number="45" name="Holes" color="7" fill="1" visible="no" active="no"/>
-<layer number="46" name="Milling" color="3" fill="1" visible="no" active="no"/>
-<layer number="47" name="Measures" color="7" fill="1" visible="no" active="no"/>
-<layer number="48" name="Document" color="7" fill="1" visible="no" active="no"/>
-<layer number="49" name="Reference" color="7" fill="1" visible="no" active="no"/>
-<layer number="51" name="tDocu" color="6" fill="1" visible="no" active="no"/>
-<layer number="52" name="bDocu" color="7" fill="1" visible="no" active="no"/>
+<layer number="46" name="Milling" color="3" fill="1" visible="yes" active="no"/>
+<layer number="47" name="Measures" color="7" fill="1" visible="yes" active="no"/>
+<layer number="48" name="Document" color="7" fill="1" visible="yes" active="no"/>
+<layer number="49" name="Reference" color="7" fill="1" visible="yes" active="no"/>
+<layer number="51" name="tDocu" color="7" fill="1" visible="yes" active="no"/>
+<layer number="52" name="bDocu" color="7" fill="1" visible="yes" active="no"/>
 <layer number="91" name="Nets" color="2" fill="1" visible="yes" active="yes"/>
 <layer number="92" name="Busses" color="1" fill="1" visible="yes" active="yes"/>
@@
 </classes>
 <parts>
-<part name="IC1" library="microchip" deviceset="PIC18F1*20" device="P" technology="2"/>
+<part name="IC1" library="microchip" deviceset="PIC18F1*20" device="P" technology="2">
+<attribute name="MPN" value="PIC18F1320-I/P"/>
+</part>
 <part name="IC2" library="ic-package" deviceset="DIL8" device="S" value="OX-52 10mhz"/>
 <part name="IC3" library="ic-package" deviceset="DIL16" device="S" value="LX2885IGW"/>
@@
 <part name="VSS3" library="supply1" deviceset="VSS" device=""/>
 <part name="VSS4" library="supply1" deviceset="VSS" device=""/>
+<part name="C8" library="resistor" deviceset="C-US" device="025-024X044" value="22"/>
+<part name="VSS5" library="supply1" deviceset="VSS" device=""/>
 </parts>
 <sheets>
@@
 <instance part="VSS3" gate="G$1" x="111.76" y="22.86"/>
 <instance part="VSS4" gate="G$1" x="45.72" y="-22.86"/>
+<instance part="C8" gate="G$1" x="55.88" y="78.74"/>
+<instance part="VSS5" gate="G$1" x="55.88" y="71.12"/>
 </instances>
 <busses>
@@
 <pinref part="VDD1" gate="G$1" pin="VDD"/>
 <junction x="104.14" y="-5.08"/>
+<pinref part="C8" gate="G$1" pin="1"/>
+<junction x="55.88" y="81.28"/>
 </segment>
 <segment>
@@
 <junction x="35.56" y="-20.32"/>
 </segment>
-</net>
+<segment>
+<pinref part="C8" gate="G$1" pin="2"/>
+<pinref part="VSS5" gate="G$1" pin="VSS"/>
+</segment>
+</net>

Commit message: up
Parts:
- removed C8: 22, resistor:C-US025-024X044
- removed D1: HFBR1528, opto-transmittter-hp:HFBR1528
- removed D2: HFBR2528, opto-transmittter-hp:HFBR2528
- removed IC3: LX2885IGW, ic-package:DIL16S
- removed R10, R3, R4, R5, R9: 510, resistor:R-US_0204/2V
- removed R6: 10000, resistor:R-US_0204/2V
- removed R7: 2200, resistor:R-US_0204/2V
- removed R8: 100, resistor:R-US_0204/2V
- added C9: 0.1, rcl:C-USC0805
- C1, C7: value 22 -> 22uf; device resistor:C-US025-024X044 -> rcl:C-USC0805
- C2, C3, C4, C5: device resistor:C-US050-025X075 -> rcl:C-USC0805
- C6: value 0.1 -> 22uf; device resistor:C-US050-025X075 -> rcl:C-USC0805
- R1: value 510 -> 300; device resistor:R-US_0204/2V -> rcl:R-US_R0805
- R2: value 510 -> 10000; device resistor:R-US_0204/2V -> rcl:R-US_R0805
Connections:
- removed net N$1: IC3.1, R1.2
- removed net N$11: IC1.INT0/AN4/RB0, IC3.10
- removed net N$14: D1.C, IC1.INT1/CK/TX/AN5/RB1
- removed net N$16: IC1.RA0/AN0, R1.1
- removed net N$17: IC1.RA1/AN1/LVDIN, IC3.2
- removed net N$18: IC1.RA2/AN2/VREF-, R2.1
- removed net N$19: IC1.RA3/AN3/VREF+, IC3.3
- removed net N$2: IC3.4, R2.2
- removed net N$22: IC1.RA6/CLKO/OSC2, R4.2
- removed net N$23: IC1.P1A/CCP1/RB3, IC3.14
- removed net N$24: IC1.RA4/T0CKI, IC3.8
- removed net N$26: IC3.9, R10.1
- removed net N$3: IC3.16, R3.1
- removed net N$4: IC3.13, R4.1
- removed net N$7: D2.VO, IC1.BKI0/DT/RX/AN6/RB4, R7.2
- removed net N$8: D1.A, R8.1
- removed net N$9: IC3.7, R9.2
- net N$12: now also R1.1, R2.2; no longer R5.1, R6.2
- net N$20: no longer R3.2
- net N$21: no longer IC3.15
- net N$5: now also R1.2; no longer R5.2
- net VDD: now also C9.2, R2.1; no longer C8.1, D2.VCC, R10.2, R6.1, R7.1, R8.2, R9.1
- net VSS: now also C9.1; no longer C8.2, D1.GND, D1.GND@1, D2.1, D2.4, D2.GND
Other:
- moved on the sheet: C4, C6, C7, R1, R2

Commit message: up
Parts:
- added ANALOG_OUT: CC MODE SIGNAL, con-molex:22-23-2021
- added C10: 0.1, rcl:C-USC0805
- added C11, C8: 22uf, rcl:C-USC0805
- added IC3: ADM3095EBRZ, SamacSys_Parts:ADM3095EBRZ
- added JP2: RS485, pinhead:PINHD-1X6
- added L1: 10uh, rcl:L-US0204/7
- added LED1: DATA, led:LEDCHIPLED_0805
- added R3: 300, rcl:R-US_R0805
- added R4: 10000, rcl:R-US_R0805
- added R5: 2.2k, rcl:R-US_R0805
Connections:
- new net N$1: IC1.BKI0/DT/RX/AN6/RB4, IC3.RXD
- new net N$11: ANALOG_OUT-1.S, C11.1, L1.2, R4.1
- new net N$13: LED1.A, R5.1
- new net N$14: IC1.RA4/T0CKI, R5.2
- new net N$2: IC1.INT1/CK/TX/AN5/RB1, IC3.TXD
- new net N$3: IC1.RA0/AN0, IC3.DE
- new net N$4: IC1.RA1/AN1/LVDIN, IC3.!RE
- new net N$6: IC1.P1A/CCP1/RB3, R3.1
- new net N$7: L1.1, R3.2
- new net N$8: IC3.B, JP2.2
- new net N$9: IC3.A, JP2.3
- net VDD: now also C10.1, C8.1, IC3.VCC, IC3.VIO, JP2.1
- net VSS: now also ANALOG_OUT-2.S, C10.2, C11.2, C8.2, IC3.GND_1, IC3.GND_2, IC3.GND_3, IC3.GND_4, IC3.GND_5, IC3.GND_6, IC3.GND_7, IC3.GND_8, JP2.4, LED1.C, R4.2
