File: ihc_mon.sch (EAGLE design)
At the start: 26 parts, among them IC1 PIC18F1220P, IC2 OX-52 10mhz, IC3 ADM3095EBRZ, X1 22-23-2021, X2 22-23-2021

Commit message: up
Parts:
- added JP3: SIG, pinhead:PINHD-1X6
- added LSP1: SE14, solpad:SE14
- added PAD1: (no value), wirepad:3,81/1,4
- added PAD2: (no value), wirepad:SMD2
- added R6: 10000, rcl:R-US_R0805
- added R8: 120, rcl:R-US_M1206
Connections:
- new net N$17: IC1.INT0/AN4/RB0, JP3.2
- new net N$18: IC1.RA2/AN2/VREF-, JP3.3
- new net N$19: IC1.RA3/AN3/VREF+, JP3.4
- new net N$22: IC1.RA6/CLKO/OSC2, JP3.5
- net N$1: now also R6.1
- net N$8: now also R8.1
- net N$9: now also R8.2
- net VDD: now also JP3.6, R6.2
- net VSS: now also JP2.5, JP2.6, JP3.1, LSP1.MP, PAD1.P, PAD2.P
Changed lines of the file:
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@@
 <part name="VSS14" library="supply1" deviceset="VSS" device=""/>
 <part name="R5" library="rcl" library_urn="urn:adsk.eagle:library:334" deviceset="R-US_" device="R0805" package3d_urn="urn:adsk.eagle:package:23553/2" value="2.2k"/>
+<part name="R6" library="rcl" library_urn="urn:adsk.eagle:library:334" deviceset="R-US_" device="R0805" package3d_urn="urn:adsk.eagle:package:23553/2" value="10000"/>
+<part name="VDD5" library="supply1" deviceset="VDD" device=""/>
+<part name="R8" library="rcl" library_urn="urn:adsk.eagle:library:334" deviceset="R-US_" device="M1206" package3d_urn="urn:adsk.eagle:package:23566/2" value="120"/>
+<part name="JP3" library="pinhead" deviceset="PINHD-1X6" device="" value="SIG"/>
+<part name="VSS15" library="supply1" deviceset="VSS" device=""/>
+<part name="VDD6" library="supply1" deviceset="VDD" device=""/>
+<part name="VSS16" library="supply1" deviceset="VSS" device=""/>
+<part name="LSP1" library="solpad" library_urn="urn:adsk.eagle:library:364" deviceset="SE14" device="" package3d_urn="urn:adsk.eagle:package:26504/1"/>
+<part name="PAD1" library="wirepad" library_urn="urn:adsk.eagle:library:412" deviceset="3,81/1,4" device="" package3d_urn="urn:adsk.eagle:package:30835/1"/>
+<part name="PAD2" library="wirepad" library_urn="urn:adsk.eagle:library:412" deviceset="SMD2" device="" package3d_urn="urn:adsk.eagle:package:30839/1"/>
+<part name="VSS17" library="supply1" deviceset="VSS" device=""/>
 </parts>
 <sheets>
@@
 <attribute name="NAME" x="-29.4386" y="34.29" size="1.778" layer="95" rot="R90"/>
 <attribute name="VALUE" x="-24.638" y="34.29" size="1.778" layer="96" rot="R90"/>
+</instance>
+<instance part="R6" gate="G$1" x="96.52" y="40.64" smashed="yes">
+<attribute name="NAME" x="92.71" y="42.1386" size="1.778" layer="95"/>
+<attribute name="VALUE" x="92.71" y="37.338" size="1.778" layer="96"/>
+</instance>
+<instance part="VDD5" gate="G$1" x="104.14" y="40.64" smashed="yes" rot="R270">
+<attribute name="VALUE" x="101.6" y="43.18" size="1.778" layer="96"/>
+</instance>
+<instance part="R8" gate="G$1" x="134.62" y="71.12" smashed="yes" rot="R90">
+<attribute name="NAME" x="133.1214" y="67.31" size="1.778" layer="95" rot="R90"/>
+<attribute name="VALUE" x="137.922" y="67.31" size="1.778" layer="96" rot="R90"/>
+</instance>
+<instance part="JP3" gate="A" x="45.72" y="-15.24" smashed="yes" rot="R270">
+<attribute name="NAME" x="56.515" y="-8.89" size="1.778" layer="95" rot="R270"/>
+<attribute name="VALUE" x="35.56" y="-8.89" size="1.778" layer="96" rot="R270"/>
+</instance>
+<instance part="VSS15" gate="G$1" x="68.58" y="-12.7" smashed="yes" rot="R90">
+<attribute name="VALUE" x="73.66" y="-15.24" size="1.778" layer="96" rot="R180"/>
+</instance>
+<instance part="VDD6" gate="G$1" x="25.4" y="-12.7" smashed="yes" rot="R90">
+<attribute name="VALUE" x="27.94" y="-15.24" size="1.778" layer="96" rot="R180"/>
+</instance>
+<instance part="VSS16" gate="G$1" x="144.78" y="63.5" smashed="yes">
+<attribute name="VALUE" x="142.24" y="58.42" size="1.778" layer="96" rot="R90"/>
+</instance>
+<instance part="LSP1" gate="1" x="127" y="17.78" smashed="yes">
+<attribute name="NAME" x="125.73" y="20.701" size="1.778" layer="95"/>
+</instance>
+<instance part="PAD1" gate="1" x="137.16" y="17.78" smashed="yes" rot="R270">
+<attribute name="NAME" x="139.0142" y="18.923" size="1.778" layer="95" rot="R270"/>
+<attribute name="VALUE" x="133.858" y="18.923" size="1.778" layer="96" rot="R270"/>
+</instance>
+<instance part="PAD2" gate="1" x="147.32" y="17.78" smashed="yes" rot="R270">
+<attribute name="NAME" x="149.1742" y="18.923" size="1.778" layer="95" rot="R270"/>
+<attribute name="VALUE" x="144.018" y="18.923" size="1.778" layer="96" rot="R270"/>
+</instance>
+<instance part="VSS17" gate="G$1" x="124.46" y="12.7" smashed="yes">
+<attribute name="VALUE" x="121.92" y="7.62" size="1.778" layer="96" rot="R90"/>
 </instance>
 </instances>
@@
 <junction x="144.78" y="88.9"/>
 <junction x="137.16" y="88.9"/>
+</segment>
+<segment>
+<pinref part="R6" gate="G$1" pin="2"/>
+<pinref part="VDD5" gate="G$1" pin="VDD"/>
+<junction x="101.6" y="40.64"/>
+</segment>
+<segment>
+<pinref part="JP3" gate="A" pin="6"/>
+<wire x1="40.64" y1="-12.7" x2="27.94" y2="-12.7" width="0.1524" layer="91"/>
+<pinref part="VDD6" gate="G$1" pin="VDD"/>
+<junction x="27.94" y="-12.7"/>
+<junction x="40.64" y="-12.7"/>
 </segment>
 </net>
@@
 <junction x="-27.94" y="25.4"/>
 </segment>
+<segment>
+<pinref part="JP3" gate="A" pin="1"/>
+<wire x1="53.34" y1="-12.7" x2="66.04" y2="-12.7" width="0.1524" layer="91"/>
+<pinref part="VSS15" gate="G$1" pin="VSS"/>
+<junction x="66.04" y="-12.7"/>
+<junction x="53.34" y="-12.7"/>
+</segment>
+<segment>
+<pinref part="JP2" gate="A" pin="6"/>
+<wire x1="144.78" y1="76.2" x2="144.78" y2="66.04" width="0.1524" layer="91"/>
+<pinref part="VSS16" gate="G$1" pin="VSS"/>
+<junction x="144.78" y="66.04"/>
+<pinref part="JP2" gate="A" pin="5"/>
+<wire x1="144.78" y1="78.74" x2="144.78" y2="76.2" width="0.1524" layer="91"/>
+<junction x="144.78" y="78.74"/>
+<junction x="144.78" y="76.2"/>
+</segment>
+<segment>
+<pinref part="PAD2" gate="1" pin="P"/>
+<wire x1="147.32" y1="15.24" x2="137.16" y2="15.24" width="0.1524" layer="91"/>
+<pinref part="VSS17" gate="G$1" pin="VSS"/>
+<junction x="124.46" y="15.24"/>
+<pinref part="LSP1" gate="1" pin="MP"/>
+<junction x="127" y="15.24"/>
+<wire x1="137.16" y1="15.24" x2="127" y2="15.24" width="0.1524" layer="91"/>
+<wire x1="127" y1="15.24" x2="124.46" y2="15.24" width="0.1524" layer="91"/>
+<pinref part="PAD1" gate="1" pin="P"/>
+<junction x="137.16" y="15.24"/>
+<junction x="147.32" y="15.24"/>
+</segment>
 </net>
 <net name="N$10" class="0">
@@
 <junction x="93.98" y="73.66"/>
 <junction x="76.2" y="40.64"/>
+<pinref part="R6" gate="G$1" pin="1"/>
+<junction x="91.44" y="40.64"/>
 </segment>
 </net>
@@
 <segment>
 <pinref part="JP2" gate="A" pin="2"/>
-<wire x1="144.78" y1="86.36" x2="134.62" y2="86.36" width="0.1524" layer="91"/>
+<wire x1="144.78" y1="86.36" x2="139.7" y2="86.36" width="0.1524" layer="91"/>
+<wire x1="139.7" y1="86.36" x2="134.62" y2="86.36" width="0.1524" layer="91"/>
 <wire x1="134.62" y1="86.36" x2="134.62" y2="83.82" width="0.1524" layer="91"/>
 <pinref part="IC3" gate="G$1" pin="B"/>
@@
 <junction x="124.46" y="83.82"/>
 <junction x="144.78" y="86.36"/>
+<wire x1="134.62" y1="66.04" x2="139.7" y2="66.04" width="0.1524" layer="91"/>
+<wire x1="139.7" y1="66.04" x2="139.7" y2="86.36" width="0.1524" layer="91"/>
+<junction x="139.7" y="86.36"/>
+<pinref part="R8" gate="G$1" pin="1"/>
+<junction x="134.62" y="66.04"/>
 </segment>
 </net>
@@
 <segment>
 <pinref part="IC3" gate="G$1" pin="A"/>
-<wire x1="124.46" y1="76.2" x2="137.16" y2="76.2" width="0.1524" layer="91"/>
+<wire x1="124.46" y1="76.2" x2="134.62" y2="76.2" width="0.1524" layer="91"/>
+<wire x1="134.62" y1="76.2" x2="137.16" y2="76.2" width="0.1524" layer="91"/>
 <wire x1="137.16" y1="76.2" x2="137.16" y2="83.82" width="0.1524" layer="91"/>
 <pinref part="JP2" gate="A" pin="3"/>
@@
 <junction x="124.46" y="76.2"/>
 <junction x="144.78" y="83.82"/>
+<pinref part="R8" gate="G$1" pin="2"/>
+<junction x="134.62" y="76.2"/>
 </segment>
 </net>
@@
 </segment>
 </net>
+<net name="N$17" class="0">
+<segment>
+<pinref part="IC1" gate="G$1" pin="INT0/AN4/RB0"/>
+<wire x1="76.2" y1="50.8" x2="78.74" y2="50.8" width="0.1524" layer="91"/>
+<wire x1="78.74" y1="50.8" x2="78.74" y2="-5.08" width="0.1524" layer="91"/>
+<wire x1="78.74" y1="-5.08" x2="50.8" y2="-5.08" width="0.1524" layer="91"/>
+<pinref part="JP3" gate="A" pin="2"/>
+<wire x1="50.8" y1="-5.08" x2="50.8" y2="-12.7" width="0.1524" layer="91"/>
+<junction x="50.8" y="-12.7"/>
+<junction x="76.2" y="50.8"/>
+</segment>
+</net>
+<net name="N$18" class="0">
+<segment>
+<pinref part="IC1" gate="G$1" pin="RA2/AN2/VREF-"/>
+<wire x1="17.78" y1="38.1" x2="-15.24" y2="38.1" width="0.1524" layer="91"/>
+<wire x1="-15.24" y1="38.1" x2="-15.24" y2="10.16" width="0.1524" layer="91"/>
+<wire x1="-15.24" y1="10.16" x2="7.62" y2="10.16" width="0.1524" layer="91"/>
+<wire x1="7.62" y1="10.16" x2="7.62" y2="7.62" width="0.1524" layer="91"/>
+<wire x1="7.62" y1="7.62" x2="48.26" y2="7.62" width="0.1524" layer="91"/>
+<pinref part="JP3" gate="A" pin="3"/>
+<wire x1="48.26" y1="7.62" x2="48.26" y2="-12.7" width="0.1524" layer="91"/>
+<junction x="17.78" y="38.1"/>
+<junction x="48.26" y="-12.7"/>
+</segment>
+</net>
+<net name="N$19" class="0">
+<segment>
+<pinref part="IC1" gate="G$1" pin="RA3/AN3/VREF+"/>
+<wire x1="17.78" y1="35.56" x2="12.7" y2="35.56" width="0.1524" layer="91"/>
+<wire x1="12.7" y1="35.56" x2="12.7" y2="45.72" width="0.1524" layer="91"/>
+<wire x1="12.7" y1="45.72" x2="-33.02" y2="45.72" width="0.1524" layer="91"/>
+<wire x1="-33.02" y1="45.72" x2="-33.02" y2="5.08" width="0.1524" layer="91"/>
+<wire x1="-33.02" y1="5.08" x2="45.72" y2="5.08" width="0.1524" layer="91"/>
+<pinref part="JP3" gate="A" pin="4"/>
+<wire x1="45.72" y1="5.08" x2="45.72" y2="-12.7" width="0.1524" layer="91"/>
+<junction x="45.72" y="-12.7"/>
+<junction x="17.78" y="35.56"/>
+</segment>
+</net>
+<net name="N$22" class="0">
+<segment>
+<pinref part="IC1" gate="G$1" pin="RA6/CLKO/OSC2"/>
+<wire x1="17.78" y1="50.8" x2="17.78" y2="48.26" width="0.1524" layer="91"/>
+<wire x1="17.78" y1="48.26" x2="-35.56" y2="48.26" width="0.1524" layer="91"/>
+<wire x1="-35.56" y1="48.26" x2="-35.56" y2="2.54" width="0.1524" layer="91"/>
+<wire x1="-35.56" y1="2.54" x2="43.18" y2="2.54" width="0.1524" layer="91"/>
+<pinref part="JP3" gate="A" pin="5"/>
+<wire x1="43.18" y1="2.54" x2="43.18" y2="-12.7" width="0.1524" layer="91"/>
+<junction x="43.18" y="-12.7"/>
+<junction x="17.78" y="50.8"/>
+</segment>
+</net>

Commit message: up
Parts:
- added A4: a4, wirepad:SMD2
- C11: value 22uf -> 3.3uf
- GND1, GND2: value (none) -> gnd
- R3: value 300 -> 100
- R4: value 10000 -> 2200
- R5: value 2.2k -> 1000
- renumbered PAD1 to GND1, PAD2 to GND2
Connections:
- removed net N$14: IC1.RA4/T0CKI, R5.2
- new net N$16: A4.P, IC1.RA4/T0CKI
- net N$17: now also R5.2
Changed lines of the file:
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@@
 <part name="JP2" library="pinhead" deviceset="PINHD-1X6" device="" value="RS485"/>
 <part name="VDD4" library="supply1" deviceset="VDD" device=""/>
-<part name="R3" library="rcl" library_urn="urn:adsk.eagle:library:334" deviceset="R-US_" device="R0805" package3d_urn="urn:adsk.eagle:package:23553/2" value="300"/>
-<part name="C11" library="rcl" library_urn="urn:adsk.eagle:library:334" deviceset="C-US" device="C0805" package3d_urn="urn:adsk.eagle:package:23617/2" value="22uf"/>
+<part name="R3" library="rcl" library_urn="urn:adsk.eagle:library:334" deviceset="R-US_" device="R0805" package3d_urn="urn:adsk.eagle:package:23553/2" value="100"/>
+<part name="C11" library="rcl" library_urn="urn:adsk.eagle:library:334" deviceset="C-US" device="C0805" package3d_urn="urn:adsk.eagle:package:23617/2" value="3.3uf"/>
 <part name="L1" library="rcl" library_urn="urn:adsk.eagle:library:334" deviceset="L-US" device="0204/7" package3d_urn="urn:adsk.eagle:package:23498/2" value="10uh"/>
 <part name="VSS12" library="supply1" deviceset="VSS" device=""/>
-<part name="R4" library="rcl" library_urn="urn:adsk.eagle:library:334" deviceset="R-US_" device="R0805" package3d_urn="urn:adsk.eagle:package:23553/2" value="10000"/>
+<part name="R4" library="rcl" library_urn="urn:adsk.eagle:library:334" deviceset="R-US_" device="R0805" package3d_urn="urn:adsk.eagle:package:23553/2" value="2200"/>
 <part name="VSS13" library="supply1" deviceset="VSS" device=""/>
 <part name="LED1" library="led" library_urn="urn:adsk.eagle:library:259" deviceset="LED" device="CHIPLED_0805" package3d_urn="urn:adsk.eagle:package:15821/2" value="DATA"/>
 <part name="VSS14" library="supply1" deviceset="VSS" device=""/>
-<part name="R5" library="rcl" library_urn="urn:adsk.eagle:library:334" deviceset="R-US_" device="R0805" package3d_urn="urn:adsk.eagle:package:23553/2" value="2.2k"/>
+<part name="R5" library="rcl" library_urn="urn:adsk.eagle:library:334" deviceset="R-US_" device="R0805" package3d_urn="urn:adsk.eagle:package:23553/2" value="1000"/>
 <part name="R6" library="rcl" library_urn="urn:adsk.eagle:library:334" deviceset="R-US_" device="R0805" package3d_urn="urn:adsk.eagle:package:23553/2" value="10000"/>
 <part name="VDD5" library="supply1" deviceset="VDD" device=""/>
@@
 <part name="VSS16" library="supply1" deviceset="VSS" device=""/>
 <part name="LSP1" library="solpad" library_urn="urn:adsk.eagle:library:364" deviceset="SE14" device="" package3d_urn="urn:adsk.eagle:package:26504/1"/>
-<part name="PAD1" library="wirepad" library_urn="urn:adsk.eagle:library:412" deviceset="3,81/1,4" device="" package3d_urn="urn:adsk.eagle:package:30835/1"/>
-<part name="PAD2" library="wirepad" library_urn="urn:adsk.eagle:library:412" deviceset="SMD2" device="" package3d_urn="urn:adsk.eagle:package:30839/1"/>
+<part name="GND1" library="wirepad" library_urn="urn:adsk.eagle:library:412" deviceset="3,81/1,4" device="" package3d_urn="urn:adsk.eagle:package:30835/1" value="gnd"/>
+<part name="GND2" library="wirepad" library_urn="urn:adsk.eagle:library:412" deviceset="SMD2" device="" package3d_urn="urn:adsk.eagle:package:30839/1" value="gnd"/>
 <part name="VSS17" library="supply1" deviceset="VSS" device=""/>
+<part name="A4" library="wirepad" library_urn="urn:adsk.eagle:library:412" deviceset="SMD2" device="" package3d_urn="urn:adsk.eagle:package:30839/1" value="a4"/>
 </parts>
 <sheets>
@@
 <attribute name="NAME" x="125.73" y="20.701" size="1.778" layer="95"/>
 </instance>
-<instance part="PAD1" gate="1" x="137.16" y="17.78" smashed="yes" rot="R270">
+<instance part="GND1" gate="1" x="137.16" y="17.78" smashed="yes" rot="R270">
 <attribute name="NAME" x="139.0142" y="18.923" size="1.778" layer="95" rot="R270"/>
 <attribute name="VALUE" x="133.858" y="18.923" size="1.778" layer="96" rot="R270"/>
 </instance>
-<instance part="PAD2" gate="1" x="147.32" y="17.78" smashed="yes" rot="R270">
+<instance part="GND2" gate="1" x="147.32" y="17.78" smashed="yes" rot="R270">
 <attribute name="NAME" x="149.1742" y="18.923" size="1.778" layer="95" rot="R270"/>
 <attribute name="VALUE" x="144.018" y="18.923" size="1.778" layer="96" rot="R270"/>
@@
 <instance part="VSS17" gate="G$1" x="124.46" y="12.7" smashed="yes">
 <attribute name="VALUE" x="121.92" y="7.62" size="1.778" layer="96" rot="R90"/>
+</instance>
+<instance part="A4" gate="1" x="-15.24" y="43.18" smashed="yes">
+<attribute name="NAME" x="-16.383" y="45.0342" size="1.778" layer="95"/>
+<attribute name="VALUE" x="-16.383" y="39.878" size="1.778" layer="96"/>
 </instance>
 </instances>
@@
 </segment>
 <segment>
-<pinref part="PAD2" gate="1" pin="P"/>
+<pinref part="GND2" gate="1" pin="P"/>
 <wire x1="147.32" y1="15.24" x2="137.16" y2="15.24" width="0.1524" layer="91"/>
 <pinref part="VSS17" gate="G$1" pin="VSS"/>
@@
 <wire x1="137.16" y1="15.24" x2="127" y2="15.24" width="0.1524" layer="91"/>
 <wire x1="127" y1="15.24" x2="124.46" y2="15.24" width="0.1524" layer="91"/>
-<pinref part="PAD1" gate="1" pin="P"/>
+<pinref part="GND1" gate="1" pin="P"/>
 <junction x="137.16" y="15.24"/>
 <junction x="147.32" y="15.24"/>
@@
 </segment>
 </net>
-<net name="N$14" class="0">
-<segment>
-<pinref part="IC1" gate="G$1" pin="RA4/T0CKI"/>
-<wire x1="17.78" y1="33.02" x2="10.16" y2="33.02" width="0.1524" layer="91"/>
-<wire x1="10.16" y1="33.02" x2="10.16" y2="35.56" width="0.1524" layer="91"/>
-<wire x1="10.16" y1="35.56" x2="-17.78" y2="35.56" width="0.1524" layer="91"/>
-<wire x1="-17.78" y1="35.56" x2="-17.78" y2="43.18" width="0.1524" layer="91"/>
-<pinref part="R5" gate="G$1" pin="2"/>
-<wire x1="-17.78" y1="43.18" x2="-27.94" y2="43.18" width="0.1524" layer="91"/>
-<junction x="-27.94" y="43.18"/>
-<junction x="17.78" y="33.02"/>
-</segment>
-</net>
 <net name="N$17" class="0">
 <segment>
@@
 <junction x="50.8" y="-12.7"/>
 <junction x="76.2" y="50.8"/>
+<pinref part="R5" gate="G$1" pin="2"/>
+<wire x1="-27.94" y1="43.18" x2="-22.86" y2="43.18" width="0.1524" layer="91"/>
+<wire x1="-22.86" y1="43.18" x2="-22.86" y2="0" width="0.1524" layer="91"/>
+<wire x1="-22.86" y1="0" x2="50.8" y2="0" width="0.1524" layer="91"/>
+<wire x1="50.8" y1="0" x2="50.8" y2="-5.08" width="0.1524" layer="91"/>
+<junction x="50.8" y="-5.08"/>
+<junction x="-27.94" y="43.18"/>
 </segment>
 </net>
@@
 </segment>
 </net>
+<net name="N$16" class="0">
+<segment>
+<pinref part="IC1" gate="G$1" pin="RA4/T0CKI"/>
+<wire x1="17.78" y1="33.02" x2="10.16" y2="33.02" width="0.1524" layer="91"/>
+<wire x1="10.16" y1="33.02" x2="10.16" y2="35.56" width="0.1524" layer="91"/>
+<wire x1="10.16" y1="35.56" x2="-12.7" y2="35.56" width="0.1524" layer="91"/>
+<wire x1="-12.7" y1="35.56" x2="-12.7" y2="43.18" width="0.1524" layer="91"/>
+<pinref part="A4" gate="1" pin="P"/>
+</segment>
+</net>

Commit message: up
Parts:
- removed IC2: OX-52 10mhz, ic-package:DIL8S
- removed L1: 10uh, rcl:L-US0204/7
- added L2: 100uh, inductor-neosid:SM-1206
- added LED2: DATA, led:LEDCHIPLED_1206
- added OS1: 10MHz, IQD-Frequency-Products:OSC-OE-CFPS-32
- added R7: 1000, rcl:R-US_R0805
- added R9: 300, rcl:R-US_R0805
- LED1: value DATA -> POWER; device led:LEDCHIPLED_0805 -> led:LEDCHIPLED_1206
Connections:
- new net N$14: LED1.A, R7.1
- new net N$23: C2.1, R1.1, R2.2, R9.2
- net N$11: now also L2.2; no longer L1.2
- net N$12: now also R9.1; no longer C2.1, R1.1, R2.2
- net N$13: now also LED2.A; no longer LED1.A
- net N$25: now also OS1.OUT; no longer IC2.5
- net N$7: now also L2.1; no longer L1.1
- net VDD: now also OS1.CON, OS1.VDD, R7.2; no longer IC2.1, IC2.8
- net VSS: now also LED2.C, OS1.VSS; no longer IC2.4
Other:
- moved on the sheet: LED1

Commit message: up
Parts:
- R5, R7: value 1000 -> 1.47k
Changed lines of the file:
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@@
 <part name="VSS13" library="supply1" deviceset="VSS" device=""/>
 <part name="VSS14" library="supply1" deviceset="VSS" device=""/>
-<part name="R5" library="rcl" library_urn="urn:adsk.eagle:library:334" deviceset="R-US_" device="R0805" package3d_urn="urn:adsk.eagle:package:23553/2" value="1000"/>
+<part name="R5" library="rcl" library_urn="urn:adsk.eagle:library:334" deviceset="R-US_" device="R0805" package3d_urn="urn:adsk.eagle:package:23553/2" value="1.47k"/>
 <part name="R6" library="rcl" library_urn="urn:adsk.eagle:library:334" deviceset="R-US_" device="R0805" package3d_urn="urn:adsk.eagle:package:23553/2" value="10000"/>
 <part name="VDD5" library="supply1" deviceset="VDD" device=""/>
@@
 <part name="OS1" library="IQD-Frequency-Products" library_urn="urn:adsk.eagle:library:90" deviceset="OSC-OE" device="-CFPS-32" package3d_urn="urn:adsk.eagle:package:3365/1" value="10MHz"/>
 <part name="LED2" library="led" library_urn="urn:adsk.eagle:library:259" deviceset="LED" device="CHIPLED_1206" package3d_urn="urn:adsk.eagle:package:15823/2" value="DATA"/>
-<part name="R7" library="rcl" library_urn="urn:adsk.eagle:library:334" deviceset="R-US_" device="R0805" package3d_urn="urn:adsk.eagle:package:23553/2" value="1000"/>
+<part name="R7" library="rcl" library_urn="urn:adsk.eagle:library:334" deviceset="R-US_" device="R0805" package3d_urn="urn:adsk.eagle:package:23553/2" value="1.47k"/>
 <part name="LED1" library="led" library_urn="urn:adsk.eagle:library:259" deviceset="LED" device="CHIPLED_1206" package3d_urn="urn:adsk.eagle:package:15823/2" value="POWER"/>
 <part name="VSS18" library="supply1" deviceset="VSS" device=""/>
