File: pic32mk.brd (EAGLE design)
At the start: 160 x 100 mm, 1 part, among them IC1 PIC32MK1024MCF100-I_PT

Commit message: up
Parts:
- added C1, C2, C3, C4: 0.1, rcl:C0805
- added IC2: ADM3095EBRZ, SamacSys_Parts:SOIC127P600X175-16N
- added OS1: OSC-OE-CFPS-32, IQD-Frequency-Products:7.2X5.2-4-PAD
- added R1: 1k, rcl:M0805
- added R2: 10k, rcl:M0805
- added S1: B3W-9000-Y1N, B3W-9000-Y1N:B3W-9_1-LED
Connections:
- new net +5V: C3.1, IC2.3
- new net N$1: C1.1, R1.1, R2.1, S1.4
- new net N$2: IC1.13, R1.2
- new net N$3: IC1.63, OS1.3
- new net VDD: C2.1, C4.1, IC1.16, IC1.2, IC1.37, IC1.46, IC1.86, IC2.2, OS1.1, OS1.4, R2.2
- new net VSS: C1.2, C2.2, C3.2, C4.2, IC1.15, IC1.36, IC1.45, IC1.65, IC1.75, IC1.85, IC2.1, IC2.10, IC2.12, IC2.13, IC2.15, IC2.16, IC2.8, IC2.9, OS1.2, S1.2
Routing:
- net VDD: track 0.00 -> 110.3 mm
- net N$1: track 0.00 -> 46.1 mm
- net N$3: track 0.00 -> 22.3 mm
- net +5V: track 0.00 -> 14.4 mm
- net N$2: track 0.00 -> 10.1 mm
- added copper zone on layer 1, net VSS

Commit message: up
Routing:
- net VSS: track 0.00 -> 132.7 mm, vias 0 -> 3
- net VDD: track 110.3 -> 128.0 mm
- net +5V: track 14.4 -> 14.9 mm
- added copper zone on layer 2, net VDD
- added copper zone on layer 16, net VSS
- removed copper zone on layer 1, net VSS
