File: pic32mk.brd (EAGLE design)
At the start: 160 x 100 mm, 21 parts, among them IC1 PIC32MK1024MCF100-I_PT, IC2 ADM3095EBRZ, IC3 PIC32MK1024MCF100-I_PT

Commit message: up
Parts:
- added C10, C11: 0.1, rcl:C0805
- added F1, F2: 1206L050, polyfuse-smd_10:1206L
- added IC4: MAX203ECWP, maxim:SO20L
- added R5, R6: 0, rcl:M0805
- added S3: JS202011SCQN, JS202011SCQN_fixed:SW_JS202011SCQN
- added U$1: MAX6818, MAX6818:SSOP20
- added U$2: IRLML2502TRPBF, IRLML2502TRPBF:SOT23
Connections:
- new net +3V3: F2.2
- new net GND: IC4.6, IC4.9, U$1.GND
- new net N$3: F2.1, R5.1
- new net N$9: F1.1, R6.1
- new net VCC: IC4.7, R6.2, U$1.VCC
- net +5V: now also F1.2
- net VDD: now also C10.1, C11.1, R5.2
- net VSS: now also C10.2, C11.2
Routing:
- net VCC: track 0.00 -> 176.0 mm
- net GND: track 0.00 -> 112.9 mm, vias 0 -> 2
- net VDD: track 210.0 -> 319.9 mm, vias 0 -> 3
- net +5V: track 5.35 -> 58.7 mm
- net VSS: track 317.9 -> 334.2 mm, vias 2 -> 0
- net N$9: track 0.00 -> 4.00 mm
- net N$3: track 0.00 -> 3.99 mm
- added copper zone on layer 1, net VSS
- added copper zone on layer 16, net VSS

Commit message: up
Parts:
- added SV1: ICSP1, con-lstb:MA06-1
- added SV2: ICSP2, con-lstb:MA06-1
Connections:
- new net N$11: IC3.27, SV1.4
- new net N$12: IC3.26, SV1.5
- new net N$13: IC1.27, SV2.4
- new net N$14: IC1.26, SV2.5
- net +3V3: now also SV1.3, SV2.3
- net N$2: now also SV2.1
- net N$5: now also SV1.1
- net VSS: now also SV1.2, SV2.2
Routing:
- net +3V3: track 0.00 -> 98.4 mm, vias 0 -> 1
- net N$13: track 0.00 -> 66.5 mm
- net N$14: track 0.00 -> 65.6 mm, vias 0 -> 1
- net VSS: track 334.2 -> 392.2 mm
- net N$2: track 10.1 -> 60.0 mm, vias 0 -> 1
- net N$11: track 0.00 -> 43.3 mm
- net N$12: track 0.00 -> 38.6 mm
- net N$5: track 10.6 -> 38.0 mm
- net VDD: track 319.9 -> 337.9 mm, vias 3 -> 9
- net VCC: track 176.0 -> 175.1 mm

Commit message: up
Parts:
- added C12: 0.1, rcl:C0805
- added OS2: OSC-OE-IQXO-793, IQD-Frequency-Products:2.5X2-4-PAD
Connections:
- new net N$16: IC1.74, IC3.74, OS2.3
- net VDD: now also C12.1, OS2.1, OS2.4
- net VSS: now also C12.2, OS2.2
Routing:
- net N$16: track 0.00 -> 67.3 mm, vias 0 -> 2
- net N$14: track 65.6 -> 59.0 mm
- net N$2: track 60.0 -> 56.9 mm
- net VDD: track 337.9 -> 334.9 mm, vias 9 -> 10
- net N$13: track 66.5 -> 69.4 mm
- net N$5: track 38.0 -> 40.2 mm
- net GND: track 113.3 -> 114.1 mm
- net VSS: track 392.2 -> 391.7 mm

Commit message: up
Parts:
- moved S2 1.27 mm to (49.5, 74.9)
Connections:
- new net IC1_RPB10/PWM3H/PMPD0/RB10: IC1.93, IC3.93
- new net IC1_RPB11/PWM9H/PWM3L/PMPD1/RB11: IC1.94, IC3.94
- new net IC1_RPB12/PWM2H/PMPD2/RB12: IC1.98, IC3.98
- new net IC1_RPB13/PWM8H/PWM2L/CTPLS/PMPD3/RB13: IC1.99, IC3.99
- new net IC1_RPB14/PWM1H/VBUSON1/PMPD6/RB14: IC1.4, IC3.4
- new net IC1_RPB15/PWM7H/PWM1L/PMPD7/RB15: IC1.5, IC3.5
- new net IC1_TCK/RPA7/PWM10H/PWM4L/PMPD5/RA7: IC1.3, IC3.3
- new net IC1_TDO/PWM4H/PMPD4/RA10: IC1.100, IC3.100
Routing:
- net VSS: track 391.7 -> 0.00 mm
- net VDD: track 334.9 -> 0.00 mm, vias 10 -> 0
- net VCC: track 175.1 -> 0.00 mm
- net GND: track 114.1 -> 0.00 mm, vias 2 -> 0
- net +3V3: track 98.4 -> 0.00 mm, vias 1 -> 0
- net N$13: track 69.4 -> 0.00 mm
- net N$16: track 67.3 -> 0.00 mm, vias 2 -> 0
- net N$14: track 59.0 -> 0.00 mm, vias 1 -> 0
- net +5V: track 58.8 -> 0.00 mm
- net N$2: track 56.9 -> 0.00 mm, vias 1 -> 0
- net N$11: track 43.3 -> 0.00 mm
- net N$5: track 40.2 -> 0.00 mm
- net N$7: track 38.6 -> 0.00 mm
- net N$12: track 38.6 -> 0.00 mm
- net N$4: track 23.5 -> 0.00 mm
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
Commit message: up
Parts:
- added TP4, TP5, TP6, TP7, TP8: TPB1,27, testpad:B1,27
Connections:
- net IC1_RPB10/PWM3H/PMPD0/RB10: now also TP8.TP
- net IC1_RPB11/PWM9H/PWM3L/PMPD1/RB11: now also TP7.TP
- net IC1_RPB12/PWM2H/PMPD2/RB12: now also TP6.TP
- net IC1_RPB13/PWM8H/PWM2L/CTPLS/PMPD3/RB13: now also TP5.TP
- net IC1_RPB14/PWM1H/VBUSON1/PMPD6/RB14: no longer IC3.4
- net IC1_RPB15/PWM7H/PWM1L/PMPD7/RB15: no longer IC3.5
- net IC1_TCK/RPA7/PWM10H/PWM4L/PMPD5/RA7: no longer IC3.3
- net IC1_TDO/PWM4H/PMPD4/RA10: now also TP4.TP
Routing:
- net VSS: track 0.00 -> 372.5 mm, vias 0 -> 2
- net VDD: track 0.00 -> 324.9 mm, vias 0 -> 9
- net VCC: track 0.00 -> 178.8 mm
- net GND: track 0.00 -> 112.5 mm, vias 0 -> 2
- net +3V3: track 0.00 -> 101.5 mm, vias 0 -> 1
- net N$2: track 0.00 -> 84.3 mm
- net N$13: track 0.00 -> 69.4 mm, vias 0 -> 1
- net N$16: track 0.00 -> 67.3 mm, vias 0 -> 2
- net N$14: track 0.00 -> 63.6 mm, vias 0 -> 1
- net +5V: track 0.00 -> 58.8 mm
- net N$11: track 0.00 -> 41.5 mm, vias 0 -> 1
- net N$7: track 0.00 -> 38.6 mm
- net IC1_RPB12/PWM2H/PMPD2/RB12: track 0.00 -> 38.2 mm, vias 0 -> 2
- net N$5: track 0.00 -> 38.0 mm
- net N$12: track 0.00 -> 36.3 mm, vias 0 -> 1
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
Commit message: up
Parts:
- removed TP5, TP6, TP7, TP8: TPB1,27, testpad:B1,27
- added TP1, TP2, TP3: TPB1,27, testpad:B1,27
- moved SV2 62.0 mm to (47.0, 38.1)
- moved SV1 30.7 mm to (47.0, 64.8)
- moved OS2 10.9 mm to (108.0, 64.8), turned to 90 degrees
- moved C12 9.92 mm to (111.8, 64.8), turned to 90 degrees
- moved C2 9.67 mm to (99.1, 64.8)
- moved C4 9.67 mm to (102.9, 64.8)
- moved TP4 9.25 mm to (81.3, 58.4)
- moved OS1 8.52 mm to (92.7, 64.8)
- moved L1 5.08 mm to (78.7, 36.8), turned to 270 degrees
- moved L2 5.08 mm to (78.7, 66.0), turned to 270 degrees
- moved C6 2.54 mm to (81.3, 36.8), turned to 270 degrees
- moved C8 2.54 mm to (81.3, 66.0), turned to 270 degrees
- moved C7 1.27 mm to (83.8, 36.8), turned to 270 degrees
- moved C9 1.27 mm to (83.8, 66.0), turned to 270 degrees
Connections:
- removed net IC1_RPB14/PWM1H/VBUSON1/PMPD6/RB14: IC1.4
- removed net IC1_RPB15/PWM7H/PWM1L/PMPD7/RB15: IC1.5
- removed net IC1_TCK/RPA7/PWM10H/PWM4L/PMPD5/RA7: IC1.3
- new net N$10: IC1.3, IC3.3
- new net N$15: IC1.4, IC3.4
- new net N$17: IC1.5, IC3.5
- net IC1_RPB10/PWM3H/PMPD0/RB10: no longer TP8.TP
- net IC1_RPB11/PWM9H/PWM3L/PMPD1/RB11: no longer TP7.TP
- net IC1_RPB12/PWM2H/PMPD2/RB12: no longer TP6.TP
- net IC1_RPB13/PWM8H/PWM2L/CTPLS/PMPD3/RB13: no longer TP5.TP
- net IC1_TDO/PWM4H/PMPD4/RA10: no longer TP4.TP
- net VDD: now also IC1.62, IC3.62, TP1.TP, TP2.TP
- net VSS: now also TP3.TP, TP4.TP
Routing:
- net VSS: track 372.5 -> 175.8 mm, vias 2 -> 6
- net +3V3: track 101.5 -> 51.2 mm, vias 1 -> 0
- net N$2: track 84.3 -> 38.9 mm
- net N$13: track 69.4 -> 32.5 mm, vias 1 -> 0
- net N$14: track 63.6 -> 27.6 mm, vias 1 -> 0
- net N$15: track 0.00 -> 32.3 mm, vias 0 -> 2
- net N$17: track 0.00 -> 32.1 mm, vias 0 -> 2
- net N$10: track 0.00 -> 32.0 mm, vias 0 -> 2
- net VDD: track 324.9 -> 346.1 mm, vias 9 -> 2
- net N$16: track 67.3 -> 48.6 mm, vias 2 -> 0
- net N$5: track 38.0 -> 47.2 mm, vias 0 -> 2
- net IC1_RPB12/PWM2H/PMPD2/RB12: track 38.2 -> 29.6 mm
- net N$11: track 41.5 -> 33.5 mm, vias 1 -> 0
- net N$12: track 36.3 -> 28.7 mm, vias 1 -> 0
- net IC1_RPB11/PWM9H/PWM3L/PMPD1/RB11: track 34.7 -> 29.3 mm, vias 0 -> 2
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- added copper zone on layer 1, net VDD
- added copper zone on layer 15, net VDD
- added copper zone on layer 2, net VSS

Commit message: up
Parts:
- added TP5, TP6, TP7: TPB1,27, testpad:B1,27
Connections:
- net VDD: now also TP5.TP, TP6.TP, TP7.TP
Routing:
- net N$17: track 32.1 -> 0.00 mm, vias 2 -> 0
- net VDD: track 346.1 -> 333.7 mm, vias 2 -> 3
- net N$5: track 47.2 -> 40.7 mm

Commit message: up
Parts:
- removed C5, C8, C9: 0.1, rcl:C0805
- removed L2: 1000, inductor-neosid:SM-1206
- removed R3: 1k, rcl:M0805
- removed R4: 10k, rcl:M0805
- removed S2: B3W-9000-Y1N, B3W-9000-Y1N:B3W-9_1-LED
- removed SV1: ICSP1, con-lstb:MA06-1
- removed TP2, TP3, TP5, TP6, TP7: TPB1,27, testpad:B1,27
- added IC5: MC33931EK, MC33931EK:SOP65P1030X245-33N
- IC3: value PIC32MK1024MCF100-I_PT -> MC33931EK; device PIC32MK1024MCF100-I_PT:QFP40P1400X1400X120-100N -> MC33931EK:SOP65P1030X245-33N
- moved IC3 113.4 mm to (6.35, -6.35)
Connections:
- removed net IC1_RPB10/PWM3H/PMPD0/RB10: IC1.93, IC3.93
- removed net IC1_RPB11/PWM9H/PWM3L/PMPD1/RB11: IC1.94, IC3.94
- removed net IC1_RPB12/PWM2H/PMPD2/RB12: IC1.98, IC3.98
- removed net IC1_RPB13/PWM8H/PWM2L/CTPLS/PMPD3/RB13: IC1.99, IC3.99
- removed net IC1_TDO/PWM4H/PMPD4/RA10: IC1.100, IC3.100
- removed net N$10: IC1.3, IC3.3
- removed net N$11: IC3.27, SV1.4
- removed net N$12: IC3.26, SV1.5
- removed net N$15: IC1.4, IC3.4
- removed net N$17: IC1.5, IC3.5
- removed net N$4: C5.1, R3.1, R4.1, S2.4
- removed net N$5: IC3.13, R3.2, SV1.1
- removed net N$8: C8.1, IC3.30, L2.2
- net +3V3: no longer SV1.3
- net N$16: no longer IC3.74
- net N$7: no longer IC3.63
- net VDD: no longer C9.1, IC3.16, IC3.2, IC3.37, IC3.46, IC3.55, IC3.62, IC3.86, L2.1, R4.2, TP2.TP, TP5.TP, TP6.TP, TP7.TP
- net VSS: no longer C5.2, C8.2, C9.2, IC3.15, IC3.31, IC3.36, IC3.45, IC3.65, IC3.75, IC3.85, S2.2, SV1.2, TP3.TP
Routing:
- net VDD: track 333.7 -> 0.00 mm, vias 3 -> 0
- net VCC: track 181.4 -> 0.00 mm
- net VSS: track 175.8 -> 0.00 mm, vias 6 -> 0
- net GND: track 112.1 -> 0.00 mm, vias 2 -> 0
- net +5V: track 58.8 -> 0.00 mm
- net +3V3: track 51.2 -> 0.00 mm
- net N$16: track 48.6 -> 0.00 mm
- net N$5: track 40.7 -> 0.00 mm, vias 2 -> 0
- net N$2: track 38.9 -> 0.00 mm
- net N$7: track 34.5 -> 0.00 mm
- net N$11: track 33.5 -> 0.00 mm
- net N$13: track 32.5 -> 0.00 mm
- net IC1_RPB13/PWM8H/PWM2L/CTPLS/PMPD3/RB13: track 32.1 -> 0.00 mm, vias 2 -> 0
- net N$10: track 31.9 -> 0.00 mm, vias 2 -> 0
- net N$15: track 31.8 -> 0.00 mm, vias 2 -> 0
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- removed copper zone on layer 15, net VDD
- removed copper zone on layer 1, net VSS
- removed copper zone on layer 16, net VSS
- removed copper zone on layer 2, net VSS
