File: pic32mk.sch (EAGLE design)
At the start: 1 part, among them IC1 PIC32MK1024MCF100-I_PT

Commit message: up
Parts:
- added C1, C2, C3, C4: 0.1, rcl:C-USC0805
- added IC2: ADM3095EBRZ, SamacSys_Parts:ADM3095EBRZ
- added OS1: OSC-OE-CFPS-32, IQD-Frequency-Products:OSC-OE-CFPS-32
- added R1: 1k, rcl:R-US_M0805
- added R2: 10k, rcl:R-US_M0805
- added S1: B3W-9000-Y1N, B3W-9000-Y1N:B3W-9000-Y1N
Connections:
- new net +5V: C3.1, IC2.VIO
- new net N$1: C1.1, R1.1, R2.1, S1.4
- new net N$2: IC1.!MCLR, R1.2
- new net N$3: IC1.OSCI/CLKI/AN49/CVD49/RPC12/RC12, OS1.OUT
- new net VDD: C2.1, C4.1, IC1.VDD_1, IC1.VDD_2, IC1.VDD_3, IC1.VDD_4, IC1.VDD_6, IC2.VCC, OS1.CON, OS1.VDD, R2.2
- new net VSS: C1.2, C2.2, C3.2, C4.2, IC1.VSS_1, IC1.VSS_2, IC1.VSS_3, IC1.VSS_4, IC1.VSS_5, IC1.VSS_6, IC2.GND_1, IC2.GND_2, IC2.GND_3, IC2.GND_4, IC2.GND_5, IC2.GND_6, IC2.GND_7, IC2.GND_8, OS1.VSS, S1.2

Commit message: up
Parts:
- added C5, C6, C7, C8, C9: 0.1, rcl:C-USC0805
- added IC3: PIC32MK1024MCF100-I_PT, PIC32MK1024MCF100-I_PT:PIC32MK1024MCF100-I_PT
- added L1, L2: 1000, inductor-neosid:SM-1206
- added R3: 1k, rcl:R-US_M0805
- added R4: 10k, rcl:R-US_M0805
- added S2: B3W-9000-Y1N, B3W-9000-Y1N:B3W-9000-Y1N
Connections:
- removed net N$3: IC1.OSCI/CLKI/AN49/CVD49/RPC12/RC12, OS1.OUT
- new net N$4: C5.1, R3.1, R4.1, S2.4
- new net N$5: IC3.!MCLR, R3.2
- new net N$6: C6.1, IC1.AVDD, L1.2
- new net N$7: IC1.OSCI/CLKI/AN49/CVD49/RPC12/RC12, IC3.OSCI/CLKI/AN49/CVD49/RPC12/RC12, OS1.OUT
- new net N$8: C8.1, IC3.AVDD, L2.2
- net VDD: now also C7.1, C9.1, IC1.VUSB3V3, IC3.VDD_1, IC3.VDD_2, IC3.VDD_3, IC3.VDD_4, IC3.VDD_6, IC3.VUSB3V3, L1.1, L2.1, R4.2
- net VSS: now also C5.2, C6.2, C7.2, C8.2, C9.2, IC1.AVSS, IC3.AVSS, IC3.VSS_1, IC3.VSS_2, IC3.VSS_3, IC3.VSS_4, IC3.VSS_5, IC3.VSS_6, S2.2

Commit message: up
Parts:
- added C10, C11: 0.1, rcl:C-USC0805
- added F1, F2: 1206L050, polyfuse-smd_10:1206L050
- added IC4: MAX203ECWP, maxim:MAX203ECWP
- added R5, R6: 0, rcl:R-US_M0805
- added S3: JS202011SCQN, JS202011SCQN_fixed:JS202011SCQN
- added U$1: MAX6818, MAX6818:MAX6818
- added U$2: IRLML2502TRPBF, IRLML2502TRPBF:IRLML2502TRPBF
Connections:
- new net +3V3: F2.2
- new net GND: U$1.GND
- new net N$3: F2.1, R5.1
- new net N$9: F1.1, R6.1
- new net VCC: R6.2, U$1.VCC
- net +5V: now also F1.2
- net VDD: now also C10.1, C11.1, R5.2
- net VSS: now also C10.2, C11.2
Changed lines of the file:
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@@
 <?xml version="1.0" encoding="utf-8"?>
 <!DOCTYPE eagle SYSTEM "eagle.dtd">
-<eagle version="9.5.2">
+<eagle version="9.6.0">
 <drawing>
 <settings>
@@
 <class number="0" name="default" width="0" drill="0">
 </class>
-<class number="1" name="icurrent" width="0" drill="0">
+<class number="1" name="icurrent" width="0.0127" drill="0">
 </class>
 </classes>
@@
 <part name="VDD14" library="supply1" library_urn="urn:adsk.eagle:library:371" deviceset="VDD" device=""/>
 <part name="VDD15" library="supply1" library_urn="urn:adsk.eagle:library:371" deviceset="VDD" device=""/>
+<part name="IC4" library="maxim" library_urn="urn:adsk.eagle:library:269" deviceset="MAX203ECWP" device="" package3d_urn="urn:adsk.eagle:package:17520/2"/>
+<part name="U$1" library="MAX6818" deviceset="MAX6818" device=""/>
+<part name="U$2" library="IRLML2502TRPBF" deviceset="IRLML2502TRPBF" device=""/>
+<part name="S3" library="JS202011SCQN_fixed" deviceset="JS202011SCQN" device=""/>
+<part name="F1" library="polyfuse-smd_10" deviceset="?" device="1206L" technology="050"/>
+<part name="F2" library="polyfuse-smd_10" deviceset="?" device="1206L" technology="050"/>
+<part name="R5" library="rcl" library_urn="urn:adsk.eagle:library:334" deviceset="R-US_" device="M0805" package3d_urn="urn:adsk.eagle:package:23556/2" value="0"/>
+<part name="R6" library="rcl" library_urn="urn:adsk.eagle:library:334" deviceset="R-US_" device="M0805" package3d_urn="urn:adsk.eagle:package:23556/2" value="0"/>
+<part name="VSS24" library="supply1" library_urn="urn:adsk.eagle:library:371" deviceset="VSS" device=""/>
+<part name="VDD16" library="supply1" library_urn="urn:adsk.eagle:library:371" deviceset="VDD" device=""/>
+<part name="P+2" library="supply1" library_urn="urn:adsk.eagle:library:371" deviceset="VCC" device=""/>
+<part name="+3V1" library="supply1" library_urn="urn:adsk.eagle:library:371" deviceset="+3V3" device=""/>
+<part name="P+3" library="supply1" library_urn="urn:adsk.eagle:library:371" deviceset="+5V" device=""/>
+<part name="SUPPLY1" library="supply2" library_urn="urn:adsk.eagle:library:372" deviceset="GND" device=""/>
+<part name="SUPPLY2" library="supply2" library_urn="urn:adsk.eagle:library:372" deviceset="GND" device=""/>
+<part name="P+4" library="supply1" library_urn="urn:adsk.eagle:library:371" deviceset="VCC" device=""/>
+<part name="C10" library="rcl" library_urn="urn:adsk.eagle:library:334" deviceset="C-US" device="C0805" package3d_urn="urn:adsk.eagle:package:23617/2" value="0.1"/>
+<part name="C11" library="rcl" library_urn="urn:adsk.eagle:library:334" deviceset="C-US" device="C0805" package3d_urn="urn:adsk.eagle:package:23617/2" value="0.1"/>
+<part name="VSS25" library="supply1" library_urn="urn:adsk.eagle:library:371" deviceset="VSS" device=""/>
+<part name="VSS26" library="supply1" library_urn="urn:adsk.eagle:library:371" deviceset="VSS" device=""/>
 </parts>
 <sheets>
@@
 <instance part="VDD15" gate="G$1" x="180.34" y="-5.08" smashed="yes" rot="R270">
 <attribute name="VALUE" x="177.8" y="-2.54" size="1.778" layer="96"/>
+</instance>
+<instance part="IC4" gate="G$1" x="218.44" y="-104.14" smashed="yes">
+<attribute name="NAME" x="208.28" y="-85.725" size="1.778" layer="95"/>
+<attribute name="VALUE" x="208.28" y="-127" size="1.778" layer="96"/>
+</instance>
+<instance part="U$1" gate="G$1" x="-43.18" y="-101.6" smashed="yes">
+<attribute name="VALUE" x="-50.81086875" y="-88.8819" size="2.54361875" layer="96"/>
+<attribute name="NAME" x="-61.009" y="-65.942" size="1.7829" layer="95"/>
+</instance>
+<instance part="U$2" gate="G$1" x="-124.46" y="416.56" smashed="yes">
+<attribute name="VALUE" x="-135.921" y="416.56" size="1.78281875" layer="96"/>
+<attribute name="NAME" x="-135.9127" y="419.105059375" size="1.78153125" layer="95"/>
+</instance>
+<instance part="S3" gate="G$1" x="-78.74" y="411.48" smashed="yes">
+<attribute name="NAME" x="-94.0022" y="414.0237" size="1.27185" layer="95"/>
+<attribute name="VALUE" x="-93.9912" y="406.396259375" size="1.270940625" layer="96"/>
+</instance>
+<instance part="F1" gate="G$1" x="-124.46" y="391.16" smashed="yes">
+<attribute name="NAME" x="-128.27" y="393.7" size="1.778" layer="95"/>
+<attribute name="VALUE" x="-128.27" y="387.35" size="1.778" layer="96"/>
+</instance>
+<instance part="F2" gate="G$1" x="-124.46" y="368.3" smashed="yes">
+<attribute name="NAME" x="-128.27" y="370.84" size="1.778" layer="95"/>
+<attribute name="VALUE" x="-128.27" y="364.49" size="1.778" layer="96"/>
+</instance>
+<instance part="R5" gate="G$1" x="-114.3" y="368.3" smashed="yes">
+<attribute name="NAME" x="-118.11" y="369.7986" size="1.778" layer="95"/>
+<attribute name="VALUE" x="-118.11" y="364.998" size="1.778" layer="96"/>
+</instance>
+<instance part="R6" gate="G$1" x="-114.3" y="391.16" smashed="yes">
+<attribute name="NAME" x="-118.11" y="392.6586" size="1.778" layer="95"/>
+<attribute name="VALUE" x="-118.11" y="387.858" size="1.778" layer="96"/>
+</instance>
+<instance part="VSS24" gate="G$1" x="-109.22" y="345.44" smashed="yes">
+<attribute name="VALUE" x="-111.76" y="340.36" size="1.778" layer="96" rot="R90"/>
+</instance>
+<instance part="VDD16" gate="G$1" x="-109.22" y="365.76" smashed="yes" rot="R180">
+<attribute name="VALUE" x="-106.68" y="368.3" size="1.778" layer="96" rot="R270"/>
+</instance>
+<instance part="P+2" gate="VCC" x="-109.22" y="388.62" smashed="yes" rot="R180">
+<attribute name="VALUE" x="-106.68" y="391.16" size="1.778" layer="96" rot="R270"/>
+</instance>
+<instance part="+3V1" gate="G$1" x="-132.08" y="368.3" smashed="yes" rot="R90">
+<attribute name="VALUE" x="-127" y="365.76" size="1.778" layer="96" rot="R180"/>
+</instance>
+<instance part="P+3" gate="1" x="-132.08" y="391.16" smashed="yes" rot="R90">
+<attribute name="VALUE" x="-127" y="388.62" size="1.778" layer="96" rot="R180"/>
+</instance>
+<instance part="SUPPLY1" gate="GND" x="-119.38" y="345.44" smashed="yes">
+<attribute name="VALUE" x="-121.285" y="342.265" size="1.778" layer="96"/>
+</instance>
+<instance part="SUPPLY2" gate="GND" x="-43.18" y="-139.7" smashed="yes">
+<attribute name="VALUE" x="-45.085" y="-142.875" size="1.778" layer="96"/>
+</instance>
+<instance part="P+4" gate="VCC" x="-43.18" y="-63.5" smashed="yes">
+<attribute name="VALUE" x="-45.72" y="-66.04" size="1.778" layer="96" rot="R90"/>
+</instance>
+<instance part="C10" gate="G$1" x="-96.52" y="365.76" smashed="yes">
+<attribute name="NAME" x="-95.504" y="366.395" size="1.778" layer="95"/>
+<attribute name="VALUE" x="-95.504" y="361.569" size="1.778" layer="96"/>
+</instance>
+<instance part="C11" gate="G$1" x="-86.36" y="365.76" smashed="yes">
+<attribute name="NAME" x="-85.344" y="366.395" size="1.778" layer="95"/>
+<attribute name="VALUE" x="-85.344" y="361.569" size="1.778" layer="96"/>
+</instance>
+<instance part="VSS25" gate="G$1" x="-96.52" y="358.14" smashed="yes">
+<attribute name="VALUE" x="-99.06" y="353.06" size="1.778" layer="96" rot="R90"/>
+</instance>
+<instance part="VSS26" gate="G$1" x="-86.36" y="358.14" smashed="yes">
+<attribute name="VALUE" x="-88.9" y="353.06" size="1.778" layer="96" rot="R90"/>
 </instance>
 </instances>
@@
 </segment>
 </net>
-<net name="VDD" class="1">
+<net name="VDD" class="0">
 <segment>
 <pinref part="R2" gate="G$1" pin="2"/>
@@
 <junction x="160.02" y="-5.08"/>
 </segment>
-</net>
-<net name="VSS" class="1">
+<segment>
+<pinref part="R5" gate="G$1" pin="2"/>
+<pinref part="VDD16" gate="G$1" pin="VDD"/>
+<junction x="-109.22" y="368.3"/>
+<pinref part="C11" gate="G$1" pin="1"/>
+<wire x1="-86.36" y1="368.3" x2="-96.52" y2="368.3" width="0.1524" layer="91"/>
+<junction x="-86.36" y="368.3"/>
+<pinref part="C10" gate="G$1" pin="1"/>
+<junction x="-96.52" y="368.3"/>
+<wire x1="-96.52" y1="368.3" x2="-109.22" y2="368.3" width="0.1524" layer="91"/>
+</segment>
+</net>
+<net name="VSS" class="0">
 <segment>
 <pinref part="C1" gate="G$1" pin="2"/>
@@
 <junction x="48.26" y="180.34"/>
 </segment>
+<segment>
+<pinref part="C10" gate="G$1" pin="2"/>
+<pinref part="VSS25" gate="G$1" pin="VSS"/>
+<junction x="-96.52" y="360.68"/>
+</segment>
+<segment>
+<pinref part="C11" gate="G$1" pin="2"/>
+<pinref part="VSS26" gate="G$1" pin="VSS"/>
+<junction x="-86.36" y="360.68"/>
+</segment>
 </net>
 <net name="+5V" class="1">
@@
 <wire x1="185.42" y1="-58.42" x2="182.88" y2="-58.42" width="0.1524" layer="91"/>
 <junction x="185.42" y="-58.42"/>
+</segment>
+<segment>
+<pinref part="F1" gate="G$1" pin="2"/>
+<pinref part="P+3" gate="1" pin="+5V"/>
+<junction x="-129.54" y="391.16"/>
 </segment>
 </net>
@@
 </segment>
 </net>
+<net name="N$3" class="0">
+<segment>
+<pinref part="F2" gate="G$1" pin="1"/>
+<pinref part="R5" gate="G$1" pin="1"/>
+<junction x="-119.38" y="368.3"/>
+</segment>
+</net>
+<net name="N$9" class="0">
+<segment>
+<pinref part="F1" gate="G$1" pin="1"/>
+<pinref part="R6" gate="G$1" pin="1"/>
+<junction x="-119.38" y="391.16"/>
+</segment>
+</net>
+<net name="VCC" class="1">
+<segment>
+<pinref part="R6" gate="G$1" pin="2"/>
+<pinref part="P+2" gate="VCC" pin="VCC"/>
+<junction x="-109.22" y="391.16"/>
+</segment>
+<segment>
+<pinref part="U$1" gate="G$1" pin="VCC"/>
+<pinref part="P+4" gate="VCC" pin="VCC"/>
+</segment>
+</net>
+<net name="+3V3" class="1">
+<segment>
+<pinref part="F2" gate="G$1" pin="2"/>
+<pinref part="+3V1" gate="G$1" pin="+3V3"/>
+<junction x="-129.54" y="368.3"/>
+</segment>
+</net>
+<net name="GND" class="1">
+<segment>
+<pinref part="U$1" gate="G$1" pin="GND"/>
+<pinref part="SUPPLY2" gate="GND" pin="GND"/>
+</segment>
+<segment>
+<pinref part="SUPPLY1" gate="GND" pin="GND"/>
+<pinref part="VSS24" gate="G$1" pin="VSS"/>
+<wire x1="-119.38" y1="347.98" x2="-109.22" y2="347.98" width="0.1524" layer="91"/>
+<junction x="-119.38" y="347.98"/>
+<junction x="-109.22" y="347.98"/>
+</segment>
+</net>

Commit message: up
Parts:
- added SV1: ICSP1, con-lstb:MA06-1
- added SV2: ICSP2, con-lstb:MA06-1
Connections:
- new net N$11: IC3.PGED1/OA1IN-/AN5/CTCMP/C1IN1-/RTCC/RPB3/RB3, SV1.4
- new net N$12: IC3.PGEC1/OA1IN+/AN4/C1IN1+/C1IN3-/C2IN3-/RPB2/RB2, SV1.5
- new net N$13: IC1.PGED1/OA1IN-/AN5/CTCMP/C1IN1-/RTCC/RPB3/RB3, SV2.4
- new net N$14: IC1.PGEC1/OA1IN+/AN4/C1IN1+/C1IN3-/C2IN3-/RPB2/RB2, SV2.5
- net +3V3: now also SV1.3, SV2.3
- net N$2: now also SV2.1
- net N$5: now also SV1.1
- net VSS: now also SV1.2, SV2.2
Other:
- moved on the sheet: U$1
Changed lines of the file:
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@@
 <class number="0" name="default" width="0" drill="0">
 </class>
-<class number="1" name="icurrent" width="0.0127" drill="0">
+<class number="1" name="icurrent" width="0.2159" drill="0">
 </class>
 </classes>
@@
 <part name="VSS25" library="supply1" library_urn="urn:adsk.eagle:library:371" deviceset="VSS" device=""/>
 <part name="VSS26" library="supply1" library_urn="urn:adsk.eagle:library:371" deviceset="VSS" device=""/>
+<part name="SV1" library="con-lstb" library_urn="urn:adsk.eagle:library:162" deviceset="MA06-1" device="" package3d_urn="urn:adsk.eagle:package:8340/1" value="ICSP1"/>
+<part name="VSS27" library="supply1" library_urn="urn:adsk.eagle:library:371" deviceset="VSS" device=""/>
+<part name="+3V2" library="supply1" library_urn="urn:adsk.eagle:library:371" deviceset="+3V3" device=""/>
+<part name="SV2" library="con-lstb" library_urn="urn:adsk.eagle:library:162" deviceset="MA06-1" device="" package3d_urn="urn:adsk.eagle:package:8340/1" value="ICSP2"/>
+<part name="VSS28" library="supply1" library_urn="urn:adsk.eagle:library:371" deviceset="VSS" device=""/>
+<part name="+3V3" library="supply1" library_urn="urn:adsk.eagle:library:371" deviceset="+3V3" device=""/>
 </parts>
 <sheets>
@@
 <attribute name="VALUE" x="208.28" y="-127" size="1.778" layer="96"/>
 </instance>
-<instance part="U$1" gate="G$1" x="-43.18" y="-101.6" smashed="yes">
-<attribute name="VALUE" x="-50.81086875" y="-88.8819" size="2.54361875" layer="96"/>
-<attribute name="NAME" x="-61.009" y="-65.942" size="1.7829" layer="95"/>
+<instance part="U$1" gate="G$1" x="-66.04" y="-99.06" smashed="yes">
+<attribute name="VALUE" x="-73.67086875" y="-86.3419" size="2.54361875" layer="96"/>
+<attribute name="NAME" x="-83.869" y="-63.402" size="1.7829" layer="95"/>
 </instance>
 <instance part="U$2" gate="G$1" x="-124.46" y="416.56" smashed="yes">
@@
 <attribute name="VALUE" x="-121.285" y="342.265" size="1.778" layer="96"/>
 </instance>
-<instance part="SUPPLY2" gate="GND" x="-43.18" y="-139.7" smashed="yes">
-<attribute name="VALUE" x="-45.085" y="-142.875" size="1.778" layer="96"/>
-</instance>
-<instance part="P+4" gate="VCC" x="-43.18" y="-63.5" smashed="yes">
-<attribute name="VALUE" x="-45.72" y="-66.04" size="1.778" layer="96" rot="R90"/>
+<instance part="SUPPLY2" gate="GND" x="-66.04" y="-137.16" smashed="yes">
+<attribute name="VALUE" x="-67.945" y="-140.335" size="1.778" layer="96"/>
+</instance>
+<instance part="P+4" gate="VCC" x="-66.04" y="-58.42" smashed="yes">
+<attribute name="VALUE" x="-68.58" y="-60.96" size="1.778" layer="96" rot="R90"/>
 </instance>
 <instance part="C10" gate="G$1" x="-96.52" y="365.76" smashed="yes">
@@
 <instance part="VSS26" gate="G$1" x="-86.36" y="358.14" smashed="yes">
 <attribute name="VALUE" x="-88.9" y="353.06" size="1.778" layer="96" rot="R90"/>
+</instance>
+<instance part="SV1" gate="1" x="-63.5" y="200.66" smashed="yes">
+<attribute name="VALUE" x="-64.77" y="187.96" size="1.778" layer="96"/>
+<attribute name="NAME" x="-64.77" y="209.042" size="1.778" layer="95"/>
+</instance>
+<instance part="VSS27" gate="G$1" x="-48.26" y="185.42" smashed="yes">
+<attribute name="VALUE" x="-50.8" y="180.34" size="1.778" layer="96" rot="R90"/>
+</instance>
+<instance part="+3V2" gate="G$1" x="-48.26" y="213.36" smashed="yes">
+<attribute name="VALUE" x="-50.8" y="208.28" size="1.778" layer="96" rot="R90"/>
+</instance>
+<instance part="SV2" gate="1" x="-30.48" y="-96.52" smashed="yes">
+<attribute name="VALUE" x="-31.75" y="-109.22" size="1.778" layer="96"/>
+<attribute name="NAME" x="-31.75" y="-88.138" size="1.778" layer="95"/>
+</instance>
+<instance part="VSS28" gate="G$1" x="-15.24" y="-111.76" smashed="yes">
+<attribute name="VALUE" x="-17.78" y="-116.84" size="1.778" layer="96" rot="R90"/>
+</instance>
+<instance part="+3V3" gate="G$1" x="-15.24" y="-83.82" smashed="yes">
+<attribute name="VALUE" x="-17.78" y="-88.9" size="1.778" layer="96" rot="R90"/>
 </instance>
 </instances>
@@
 <pinref part="IC1" gate="G$1" pin="!MCLR"/>
 <pinref part="R1" gate="G$1" pin="2"/>
-<wire x1="12.7" y1="15.24" x2="-25.4" y2="15.24" width="0.1524" layer="91"/>
+<wire x1="12.7" y1="15.24" x2="-22.86" y2="15.24" width="0.1524" layer="91"/>
 <junction x="-25.4" y="15.24"/>
 <junction x="12.7" y="15.24"/>
-</segment>
-</net>
-<net name="VDD" class="0">
+<wire x1="-22.86" y1="15.24" x2="-25.4" y2="15.24" width="0.1524" layer="91"/>
+<wire x1="-25.4" y1="15.24" x2="-22.86" y2="15.24" width="0.1524" layer="91"/>
+<wire x1="-22.86" y1="15.24" x2="-22.86" y2="-71.12" width="0.1524" layer="91"/>
+<pinref part="SV2" gate="1" pin="1"/>
+<wire x1="-22.86" y1="-104.14" x2="2.54" y2="-104.14" width="0.1524" layer="91"/>
+<wire x1="2.54" y1="-104.14" x2="2.54" y2="-71.12" width="0.1524" layer="91"/>
+<junction x="2.54" y="-104.14"/>
+<junction x="-22.86" y="-104.14"/>
+<wire x1="-22.86" y1="-71.12" x2="2.54" y2="-71.12" width="0.1524" layer="91"/>
+<junction x="-22.86" y="15.24"/>
+</segment>
+</net>
+<net name="VDD" class="1">
 <segment>
 <pinref part="R2" gate="G$1" pin="2"/>
@@
 </segment>
 </net>
-<net name="VSS" class="0">
+<net name="VSS" class="1">
 <segment>
 <pinref part="C1" gate="G$1" pin="2"/>
@@
 <junction x="-86.36" y="360.68"/>
 </segment>
+<segment>
+<pinref part="SV1" gate="1" pin="2"/>
+<wire x1="-55.88" y1="195.58" x2="-48.26" y2="195.58" width="0.1524" layer="91"/>
+<wire x1="-48.26" y1="195.58" x2="-48.26" y2="187.96" width="0.1524" layer="91"/>
+<pinref part="VSS27" gate="G$1" pin="VSS"/>
+<junction x="-48.26" y="187.96"/>
+<junction x="-55.88" y="195.58"/>
+</segment>
+<segment>
+<pinref part="SV2" gate="1" pin="2"/>
+<wire x1="-22.86" y1="-101.6" x2="-15.24" y2="-101.6" width="0.1524" layer="91"/>
+<wire x1="-15.24" y1="-101.6" x2="-15.24" y2="-109.22" width="0.1524" layer="91"/>
+<pinref part="VSS28" gate="G$1" pin="VSS"/>
+<junction x="-15.24" y="-109.22"/>
+<junction x="-22.86" y="-101.6"/>
+</segment>
 </net>
 <net name="+5V" class="1">
@@
 <pinref part="IC3" gate="G$1" pin="!MCLR"/>
 <pinref part="R3" gate="G$1" pin="2"/>
-<wire x1="10.16" y1="312.42" x2="-33.02" y2="312.42" width="0.1524" layer="91"/>
+<wire x1="10.16" y1="312.42" x2="-27.94" y2="312.42" width="0.1524" layer="91"/>
+<junction x="10.16" y="312.42"/>
+<pinref part="SV1" gate="1" pin="1"/>
+<wire x1="-30.48" y1="312.42" x2="-33.02" y2="312.42" width="0.1524" layer="91"/>
+<wire x1="-55.88" y1="193.04" x2="-30.48" y2="193.04" width="0.1524" layer="91"/>
+<wire x1="-30.48" y1="193.04" x2="-30.48" y2="226.06" width="0.1524" layer="91"/>
+<wire x1="-30.48" y1="226.06" x2="-30.48" y2="312.42" width="0.1524" layer="91"/>
+<wire x1="-30.48" y1="312.42" x2="-27.94" y2="312.42" width="0.1524" layer="91"/>
 <junction x="-33.02" y="312.42"/>
-<junction x="10.16" y="312.42"/>
+<junction x="-30.48" y="312.42"/>
+<junction x="-30.48" y="193.04"/>
+<junction x="-55.88" y="193.04"/>
+<junction x="-30.48" y="226.06"/>
 </segment>
 </net>
@@
 <pinref part="U$1" gate="G$1" pin="VCC"/>
 <pinref part="P+4" gate="VCC" pin="VCC"/>
+<wire x1="-66.04" y1="-63.5" x2="-66.04" y2="-60.96" width="0.1524" layer="91"/>
 </segment>
 </net>
@@
 <pinref part="+3V1" gate="G$1" pin="+3V3"/>
 <junction x="-129.54" y="368.3"/>
+</segment>
+<segment>
+<pinref part="SV1" gate="1" pin="3"/>
+<wire x1="-55.88" y1="198.12" x2="-48.26" y2="198.12" width="0.1524" layer="91"/>
+<wire x1="-48.26" y1="198.12" x2="-48.26" y2="210.82" width="0.1524" layer="91"/>
+<junction x="-55.88" y="198.12"/>
+<pinref part="+3V2" gate="G$1" pin="+3V3"/>
+<junction x="-48.26" y="210.82"/>
+</segment>
+<segment>
+<pinref part="SV2" gate="1" pin="3"/>
+<wire x1="-22.86" y1="-99.06" x2="-15.24" y2="-99.06" width="0.1524" layer="91"/>
+<wire x1="-15.24" y1="-99.06" x2="-15.24" y2="-86.36" width="0.1524" layer="91"/>
+<junction x="-22.86" y="-99.06"/>
+<pinref part="+3V3" gate="G$1" pin="+3V3"/>
+<junction x="-15.24" y="-86.36"/>
 </segment>
 </net>
@@
 </segment>
 </net>
+<net name="N$11" class="0">
+<segment>
+<pinref part="SV1" gate="1" pin="4"/>
+<wire x1="-55.88" y1="200.66" x2="-10.16" y2="200.66" width="0.1524" layer="91"/>
+<pinref part="IC3" gate="G$1" pin="PGED1/OA1IN-/AN5/CTCMP/C1IN1-/RTCC/RPB3/RB3"/>
+<wire x1="-10.16" y1="200.66" x2="55.88" y2="200.66" width="0.1524" layer="91"/>
+<wire x1="55.88" y1="200.66" x2="55.88" y2="208.28" width="0.1524" layer="91"/>
+<junction x="-55.88" y="200.66"/>
+<junction x="55.88" y="208.28"/>
+<junction x="-10.16" y="200.66"/>
+</segment>
+</net>
+<net name="N$12" class="0">
+<segment>
+<pinref part="SV1" gate="1" pin="5"/>
+<wire x1="-55.88" y1="203.2" x2="-10.16" y2="203.2" width="0.1524" layer="91"/>
+<pinref part="IC3" gate="G$1" pin="PGEC1/OA1IN+/AN4/C1IN1+/C1IN3-/C2IN3-/RPB2/RB2"/>
+<wire x1="-10.16" y1="203.2" x2="53.34" y2="203.2" width="0.1524" layer="91"/>
+<wire x1="53.34" y1="203.2" x2="53.34" y2="208.28" width="0.1524" layer="91"/>
+<junction x="-55.88" y="203.2"/>
+<junction x="53.34" y="208.28"/>
+<junction x="-10.16" y="203.2"/>
+</segment>
+</net>
+<net name="N$13" class="0">
+<segment>
+<pinref part="SV2" gate="1" pin="4"/>
+<wire x1="-22.86" y1="-96.52" x2="58.42" y2="-96.52" width="0.1524" layer="91"/>
+<junction x="-22.86" y="-96.52"/>
+<pinref part="IC1" gate="G$1" pin="PGED1/OA1IN-/AN5/CTCMP/C1IN1-/RTCC/RPB3/RB3"/>
+<wire x1="58.42" y1="-88.9" x2="58.42" y2="-96.52" width="0.1524" layer="91"/>
+<junction x="58.42" y="-88.9"/>
+</segment>
+</net>
+<net name="N$14" class="0">
+<segment>
+<pinref part="SV2" gate="1" pin="5"/>
+<wire x1="-22.86" y1="-93.98" x2="55.88" y2="-93.98" width="0.1524" layer="91"/>
+<junction x="-22.86" y="-93.98"/>
+<pinref part="IC1" gate="G$1" pin="PGEC1/OA1IN+/AN4/C1IN1+/C1IN3-/C2IN3-/RPB2/RB2"/>
+<wire x1="55.88" y1="-88.9" x2="55.88" y2="-93.98" width="0.1524" layer="91"/>
+<junction x="55.88" y="-88.9"/>
+</segment>
+</net>
