File: pic32mk.sch (EAGLE design)
At the start: 33 parts, among them IC1 PIC32MK1024MCF100-I_PT, IC2 ADM3095EBRZ, IC3 PIC32MK1024MCF100-I_PT, IC4 MAX203ECWP

Commit message: up
Parts:
- added C12: 0.1, rcl:C-USC0805
- added OS2: OSC-OE-IQXO-793, IQD-Frequency-Products:OSC-OE-IQXO-793
Connections:
- new net N$16: IC1.SOSCO/RPB8(4)/RB8(4), IC3.SOSCO/RPB8(4)/RB8(4), OS2.OUT
- net VDD: now also C12.1, OS2.CON, OS2.VDD
- net VSS: now also C12.2, OS2.VSS
Changed lines of the file:
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@@
 <part name="VSS28" library="supply1" library_urn="urn:adsk.eagle:library:371" deviceset="VSS" device=""/>
 <part name="+3V3" library="supply1" library_urn="urn:adsk.eagle:library:371" deviceset="+3V3" device=""/>
+<part name="OS2" library="IQD-Frequency-Products" library_urn="urn:adsk.eagle:library:90" deviceset="OSC-OE" device="-IQXO-793" package3d_urn="urn:adsk.eagle:package:3371/1"/>
+<part name="C12" library="rcl" library_urn="urn:adsk.eagle:library:334" deviceset="C-US" device="C0805" package3d_urn="urn:adsk.eagle:package:23617/2" value="0.1"/>
+<part name="VDD17" library="supply1" library_urn="urn:adsk.eagle:library:371" deviceset="VDD" device=""/>
+<part name="VDD18" library="supply1" library_urn="urn:adsk.eagle:library:371" deviceset="VDD" device=""/>
+<part name="VSS29" library="supply1" library_urn="urn:adsk.eagle:library:371" deviceset="VSS" device=""/>
 </parts>
 <sheets>
@@
 <instance part="+3V3" gate="G$1" x="-15.24" y="-83.82" smashed="yes">
 <attribute name="VALUE" x="-17.78" y="-88.9" size="1.778" layer="96" rot="R90"/>
+</instance>
+<instance part="OS2" gate="A" x="238.76" y="45.72" smashed="yes" rot="R180">
+<attribute name="NAME" x="246.38" y="37.465" size="1.778" layer="95" rot="R180"/>
+<attribute name="VALUE" x="246.38" y="55.88" size="1.778" layer="96" rot="R180"/>
+</instance>
+<instance part="C12" gate="G$1" x="251.46" y="43.18" smashed="yes" rot="R180">
+<attribute name="NAME" x="250.444" y="42.545" size="1.778" layer="95" rot="R180"/>
+<attribute name="VALUE" x="250.444" y="47.371" size="1.778" layer="96" rot="R180"/>
+</instance>
+<instance part="VDD17" gate="G$1" x="251.46" y="38.1" smashed="yes" rot="R180">
+<attribute name="VALUE" x="254" y="40.64" size="1.778" layer="96" rot="R270"/>
+</instance>
+<instance part="VDD18" gate="G$1" x="226.06" y="38.1" smashed="yes" rot="R180">
+<attribute name="VALUE" x="228.6" y="40.64" size="1.778" layer="96" rot="R270"/>
+</instance>
+<instance part="VSS29" gate="G$1" x="251.46" y="53.34" smashed="yes" rot="R180">
+<attribute name="VALUE" x="254" y="58.42" size="1.778" layer="96" rot="R270"/>
 </instance>
 </instances>
@@
 <wire x1="-96.52" y1="368.3" x2="-109.22" y2="368.3" width="0.1524" layer="91"/>
 </segment>
+<segment>
+<pinref part="OS2" gate="A" pin="VDD"/>
+<pinref part="C12" gate="G$1" pin="1"/>
+<pinref part="VDD17" gate="G$1" pin="VDD"/>
+<junction x="251.46" y="40.64"/>
+<pinref part="VDD17" gate="G$1" pin="VDD"/>
+</segment>
+<segment>
+<pinref part="OS2" gate="A" pin="CON"/>
+<pinref part="VDD18" gate="G$1" pin="VDD"/>
+<junction x="226.06" y="40.64"/>
+</segment>
 </net>
 <net name="VSS" class="1">
@@
 <junction x="-15.24" y="-109.22"/>
 <junction x="-22.86" y="-101.6"/>
+</segment>
+<segment>
+<pinref part="OS2" gate="A" pin="VSS"/>
+<pinref part="VSS29" gate="G$1" pin="VSS"/>
+<pinref part="C12" gate="G$1" pin="2"/>
+<wire x1="251.46" y1="48.26" x2="251.46" y2="50.8" width="0.1524" layer="91"/>
+<junction x="251.46" y="48.26"/>
+<junction x="251.46" y="50.8"/>
 </segment>
 </net>
@@
 </segment>
 </net>
+<net name="N$16" class="0">
+<segment>
+<pinref part="IC3" gate="G$1" pin="SOSCO/RPB8(4)/RB8(4)"/>
+<wire x1="157.48" y1="340.36" x2="223.52" y2="340.36" width="0.1524" layer="91"/>
+<wire x1="223.52" y1="340.36" x2="223.52" y2="45.72" width="0.1524" layer="91"/>
+<pinref part="IC1" gate="G$1" pin="SOSCO/RPB8(4)/RB8(4)"/>
+<wire x1="160.02" y1="43.18" x2="226.06" y2="43.18" width="0.1524" layer="91"/>
+<pinref part="OS2" gate="A" pin="OUT"/>
+<wire x1="226.06" y1="43.18" x2="226.06" y2="45.72" width="0.1524" layer="91"/>
+<junction x="160.02" y="43.18"/>
+<junction x="226.06" y="45.72"/>
+<wire x1="223.52" y1="45.72" x2="226.06" y2="45.72" width="0.1524" layer="91"/>
+</segment>
+</net>

Commit message: up
Connections:
- new net IC1_RPB10/PWM3H/PMPD0/RB10: IC1.RPB10/PWM3H/PMPD0/RB10, IC3.RPB10/PWM3H/PMPD0/RB10
- new net IC1_RPB11/PWM9H/PWM3L/PMPD1/RB11: IC1.RPB11/PWM9H/PWM3L/PMPD1/RB11, IC3.RPB11/PWM9H/PWM3L/PMPD1/RB11
- new net IC1_RPB12/PWM2H/PMPD2/RB12: IC1.RPB12/PWM2H/PMPD2/RB12, IC3.RPB12/PWM2H/PMPD2/RB12
- new net IC1_RPB13/PWM8H/PWM2L/CTPLS/PMPD3/RB13: IC1.RPB13/PWM8H/PWM2L/CTPLS/PMPD3/RB13, IC3.RPB13/PWM8H/PWM2L/CTPLS/PMPD3/RB13
- new net IC1_RPB14/PWM1H/VBUSON1/PMPD6/RB14: IC1.RPB14/PWM1H/VBUSON1/PMPD6/RB14, IC3.RPB14/PWM1H/VBUSON1/PMPD6/RB14
- new net IC1_RPB15/PWM7H/PWM1L/PMPD7/RB15: IC1.RPB15/PWM7H/PWM1L/PMPD7/RB15, IC3.RPB15/PWM7H/PWM1L/PMPD7/RB15
- new net IC1_TCK/RPA7/PWM10H/PWM4L/PMPD5/RA7: IC1.TCK/RPA7/PWM10H/PWM4L/PMPD5/RA7, IC3.TCK/RPA7/PWM10H/PWM4L/PMPD5/RA7
- new net IC1_TDO/PWM4H/PMPD4/RA10: IC1.TDO/PWM4H/PMPD4/RA10, IC3.TDO/PWM4H/PMPD4/RA10
Changed lines of the file:
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@@
 <?xml version="1.0" encoding="utf-8"?>
 <!DOCTYPE eagle SYSTEM "eagle.dtd">
-<eagle version="9.6.0">
+<eagle version="9.6.1">
 <drawing>
 <settings>
@@
 <instances>
 <instance part="IC1" gate="G$1" x="12.7" y="45.72" smashed="yes">
-<attribute name="NAME" x="156.21" y="104.14" size="1.778" layer="95" align="center-left"/>
+<attribute name="NAME" x="156.21" y="104.14" size="1.778" layer="91" align="center-left"/>
 <attribute name="VALUE" x="156.21" y="101.6" size="1.778" layer="96" align="center-left"/>
 </instance>
@@
 </instances>
 <busses>
+<bus name="DPMP1:IC1_RPB10/PWM3H/PMPD0/RB10,IC1_RPB11/PWM9H/PWM3L/PMPD1/RB11,IC1_RPB12/PWM2H/PMPD2/RB12,IC1_RPB13/PWM8H/PWM2L/CTPLS/PMPD3/RB13,IC1_RPB14/PWM1H/VBUSON1/PMPD6/RB14,IC1_RPB15/PWM7H/PWM1L/PMPD7/RB15,IC1_TCK/RPA7/PWM10H/PWM4L/PMPD5/RA7,IC1_TDO/PWM4H/PMPD4/RA10">
+<segment>
+<wire x1="50.8" y1="482.6" x2="73.66" y2="482.6" width="0.762" layer="92"/>
+</segment>
+</bus>
 </busses>
 <nets>
@@
 <pinref part="VDD17" gate="G$1" pin="VDD"/>
 <junction x="251.46" y="40.64"/>
-<pinref part="VDD17" gate="G$1" pin="VDD"/>
 </segment>
 <segment>
@@
 <junction x="226.06" y="45.72"/>
 <wire x1="223.52" y1="45.72" x2="226.06" y2="45.72" width="0.1524" layer="91"/>
+</segment>
+</net>
+<net name="IC1_TCK/RPA7/PWM10H/PWM4L/PMPD5/RA7" class="0">
+<segment>
+<pinref part="IC1" gate="G$1" pin="TCK/RPA7/PWM10H/PWM4L/PMPD5/RA7"/>
+<wire x1="12.7" y1="40.64" x2="-50.8" y2="40.64" width="0.1524" layer="91"/>
+<label x="-48.26" y="40.64" size="1.778" layer="95"/>
+<junction x="12.7" y="40.64"/>
+</segment>
+<segment>
+<wire x1="53.34" y1="482.6" x2="-38.1" y2="396.24" width="0.1524" layer="91"/>
+<wire x1="-38.1" y1="396.24" x2="-38.1" y2="337.82" width="0.1524" layer="91"/>
+<label x="-38.1" y="340.36" size="1.778" layer="95" rot="R90"/>
+<pinref part="IC3" gate="G$1" pin="TCK/RPA7/PWM10H/PWM4L/PMPD5/RA7"/>
+<wire x1="10.16" y1="337.82" x2="-38.1" y2="337.82" width="0.1524" layer="91"/>
+<junction x="10.16" y="337.82"/>
+</segment>
+</net>
+<net name="IC1_RPB14/PWM1H/VBUSON1/PMPD6/RB14" class="0">
+<segment>
+<pinref part="IC1" gate="G$1" pin="RPB14/PWM1H/VBUSON1/PMPD6/RB14"/>
+<wire x1="12.7" y1="38.1" x2="-50.8" y2="38.1" width="0.1524" layer="91"/>
+<label x="-48.26" y="38.1" size="1.778" layer="95"/>
+<junction x="12.7" y="38.1"/>
+</segment>
+<segment>
+<wire x1="50.8" y1="482.6" x2="-45.72" y2="391.16" width="0.1524" layer="91"/>
+<wire x1="-45.72" y1="391.16" x2="-45.72" y2="335.28" width="0.1524" layer="91"/>
+<label x="-45.72" y="337.82" size="1.778" layer="95" rot="R90"/>
+<pinref part="IC3" gate="G$1" pin="RPB14/PWM1H/VBUSON1/PMPD6/RB14"/>
+<wire x1="10.16" y1="335.28" x2="-45.72" y2="335.28" width="0.1524" layer="91"/>
+<junction x="10.16" y="335.28"/>
+</segment>
+</net>
+<net name="IC1_RPB15/PWM7H/PWM1L/PMPD7/RB15" class="0">
+<segment>
+<pinref part="IC1" gate="G$1" pin="RPB15/PWM7H/PWM1L/PMPD7/RB15"/>
+<wire x1="12.7" y1="35.56" x2="-50.8" y2="35.56" width="0.1524" layer="91"/>
+<label x="-48.26" y="35.56" size="1.778" layer="95"/>
+<junction x="12.7" y="35.56"/>
+</segment>
+<segment>
+<wire x1="50.8" y1="482.6" x2="-50.8" y2="388.62" width="0.1524" layer="91"/>
+<wire x1="-50.8" y1="388.62" x2="-50.8" y2="332.74" width="0.1524" layer="91"/>
+<label x="-50.8" y="335.28" size="1.778" layer="95" rot="R90"/>
+<pinref part="IC3" gate="G$1" pin="RPB15/PWM7H/PWM1L/PMPD7/RB15"/>
+<wire x1="10.16" y1="332.74" x2="-50.8" y2="332.74" width="0.1524" layer="91"/>
+<junction x="10.16" y="332.74"/>
+</segment>
+</net>
+<net name="IC1_TDO/PWM4H/PMPD4/RA10" class="0">
+<segment>
+<pinref part="IC1" gate="G$1" pin="TDO/PWM4H/PMPD4/RA10"/>
+<wire x1="55.88" y1="104.14" x2="55.88" y2="167.64" width="0.1524" layer="91"/>
+<label x="55.88" y="162.56" size="1.778" layer="95" rot="R90" align="bottom-right"/>
+<junction x="55.88" y="104.14"/>
+</segment>
+<segment>
+<wire x1="53.34" y1="482.6" x2="53.34" y2="401.32" width="0.1524" layer="91"/>
+<label x="53.34" y="403.86" size="1.778" layer="95" rot="R90"/>
+<pinref part="IC3" gate="G$1" pin="TDO/PWM4H/PMPD4/RA10"/>
+<junction x="53.34" y="401.32"/>
+</segment>
+</net>
+<net name="IC1_RPB13/PWM8H/PWM2L/CTPLS/PMPD3/RB13" class="0">
+<segment>
+<pinref part="IC1" gate="G$1" pin="RPB13/PWM8H/PWM2L/CTPLS/PMPD3/RB13"/>
+<wire x1="58.42" y1="104.14" x2="58.42" y2="167.64" width="0.1524" layer="91"/>
+<label x="58.42" y="165.1" size="1.778" layer="95" rot="R90" align="bottom-right"/>
+<junction x="58.42" y="104.14"/>
+</segment>
+<segment>
+<wire x1="55.88" y1="482.6" x2="55.88" y2="401.32" width="0.1524" layer="91"/>
+<label x="55.88" y="403.86" size="1.778" layer="95" rot="R90"/>
+<pinref part="IC3" gate="G$1" pin="RPB13/PWM8H/PWM2L/CTPLS/PMPD3/RB13"/>
+<junction x="55.88" y="401.32"/>
+</segment>
+</net>
+<net name="IC1_RPB12/PWM2H/PMPD2/RB12" class="0">
+<segment>
+<pinref part="IC1" gate="G$1" pin="RPB12/PWM2H/PMPD2/RB12"/>
+<wire x1="60.96" y1="104.14" x2="60.96" y2="167.64" width="0.1524" layer="91"/>
+<label x="60.96" y="165.1" size="1.778" layer="95" rot="R90" align="bottom-right"/>
+<junction x="60.96" y="104.14"/>
+</segment>
+<segment>
+<wire x1="58.42" y1="482.6" x2="58.42" y2="447.04" width="0.1524" layer="91"/>
+<wire x1="58.42" y1="447.04" x2="58.42" y2="401.32" width="0.1524" layer="91"/>
+<label x="58.42" y="403.86" size="1.778" layer="95" rot="R90"/>
+<pinref part="IC3" gate="G$1" pin="RPB12/PWM2H/PMPD2/RB12"/>
+<junction x="58.42" y="401.32"/>
+</segment>
+</net>
+<net name="IC1_RPB11/PWM9H/PWM3L/PMPD1/RB11" class="0">
+<segment>
+<pinref part="IC1" gate="G$1" pin="RPB11/PWM9H/PWM3L/PMPD1/RB11"/>
+<wire x1="71.12" y1="104.14" x2="71.12" y2="167.64" width="0.1524" layer="91"/>
+<label x="71.12" y="165.1" size="1.778" layer="95" rot="R90" align="bottom-right"/>
+<junction x="71.12" y="104.14"/>
+</segment>
+<segment>
+<wire x1="71.12" y1="482.6" x2="68.58" y2="454.66" width="0.1524" layer="91"/>
+<wire x1="68.58" y1="454.66" x2="68.58" y2="401.32" width="0.1524" layer="91"/>
+<label x="68.58" y="403.86" size="1.778" layer="95" rot="R90"/>
+<pinref part="IC3" gate="G$1" pin="RPB11/PWM9H/PWM3L/PMPD1/RB11"/>
+<junction x="68.58" y="401.32"/>
+</segment>
+</net>
+<net name="IC1_RPB10/PWM3H/PMPD0/RB10" class="0">
+<segment>
+<pinref part="IC1" gate="G$1" pin="RPB10/PWM3H/PMPD0/RB10"/>
+<wire x1="73.66" y1="104.14" x2="73.66" y2="167.64" width="0.1524" layer="91"/>
+<label x="73.66" y="165.1" size="1.778" layer="95" rot="R90" align="bottom-right"/>
+<junction x="73.66" y="104.14"/>
+</segment>
+<segment>
+<wire x1="73.66" y1="482.6" x2="71.12" y2="447.04" width="0.1524" layer="91"/>
+<wire x1="71.12" y1="447.04" x2="71.12" y2="401.32" width="0.1524" layer="91"/>
+<label x="71.12" y="403.86" size="1.778" layer="95" rot="R90"/>
+<pinref part="IC3" gate="G$1" pin="RPB10/PWM3H/PMPD0/RB10"/>
+<junction x="71.12" y="401.32"/>
 </segment>
 </net>
@@
 for full support of SPICE simulation.
 </note>
+<note version="9.0" severity="warning">
+Since Version 9.0, EAGLE supports the align property for labels.
+Labels in schematic will not be understood with this version. Update EAGLE to the latest version
+for full support of labels.
+</note>
 </compatibility>

Commit message: up
Parts:
- added TP4, TP5, TP6, TP7, TP8: TPB1,27, testpad:TPB1,27
Connections:
- net IC1_RPB10/PWM3H/PMPD0/RB10: now also TP8.TP
- net IC1_RPB11/PWM9H/PWM3L/PMPD1/RB11: now also TP7.TP
- net IC1_RPB12/PWM2H/PMPD2/RB12: now also TP6.TP
- net IC1_RPB13/PWM8H/PWM2L/CTPLS/PMPD3/RB13: now also TP5.TP
- net IC1_RPB14/PWM1H/VBUSON1/PMPD6/RB14: no longer IC3.RPB14/PWM1H/VBUSON1/PMPD6/RB14
- net IC1_RPB15/PWM7H/PWM1L/PMPD7/RB15: no longer IC3.RPB15/PWM7H/PWM1L/PMPD7/RB15
- net IC1_TCK/RPA7/PWM10H/PWM4L/PMPD5/RA7: no longer IC3.TCK/RPA7/PWM10H/PWM4L/PMPD5/RA7
- net IC1_TDO/PWM4H/PMPD4/RA10: now also TP4.TP
Changed lines of the file:
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@@
 <part name="VDD18" library="supply1" library_urn="urn:adsk.eagle:library:371" deviceset="VDD" device=""/>
 <part name="VSS29" library="supply1" library_urn="urn:adsk.eagle:library:371" deviceset="VSS" device=""/>
+<part name="TP4" library="testpad" library_urn="urn:adsk.eagle:library:385" deviceset="TP" device="B1,27" package3d_urn="urn:adsk.eagle:package:27944/2"/>
+<part name="TP5" library="testpad" library_urn="urn:adsk.eagle:library:385" deviceset="TP" device="B1,27" package3d_urn="urn:adsk.eagle:package:27944/2"/>
+<part name="TP6" library="testpad" library_urn="urn:adsk.eagle:library:385" deviceset="TP" device="B1,27" package3d_urn="urn:adsk.eagle:package:27944/2"/>
+<part name="TP7" library="testpad" library_urn="urn:adsk.eagle:library:385" deviceset="TP" device="B1,27" package3d_urn="urn:adsk.eagle:package:27944/2"/>
+<part name="TP8" library="testpad" library_urn="urn:adsk.eagle:library:385" deviceset="TP" device="B1,27" package3d_urn="urn:adsk.eagle:package:27944/2"/>
 </parts>
 <sheets>
@@
 <attribute name="VALUE" x="254" y="58.42" size="1.778" layer="96" rot="R270"/>
 </instance>
+<instance part="TP4" gate="G$1" x="55.88" y="170.18" smashed="yes">
+<attribute name="NAME" x="54.61" y="171.45" size="1.778" layer="95"/>
+<attribute name="TP_SIGNAL_NAME" x="57.15" y="168.91" size="1.778" layer="97"/>
+</instance>
+<instance part="TP5" gate="G$1" x="58.42" y="170.18" smashed="yes">
+<attribute name="NAME" x="57.15" y="171.45" size="1.778" layer="95"/>
+<attribute name="TP_SIGNAL_NAME" x="59.69" y="168.91" size="1.778" layer="97"/>
+</instance>
+<instance part="TP6" gate="G$1" x="60.96" y="170.18" smashed="yes">
+<attribute name="NAME" x="59.69" y="171.45" size="1.778" layer="95"/>
+<attribute name="TP_SIGNAL_NAME" x="62.23" y="168.91" size="1.778" layer="97"/>
+</instance>
+<instance part="TP7" gate="G$1" x="71.12" y="170.18" smashed="yes">
+<attribute name="NAME" x="69.85" y="171.45" size="1.778" layer="95"/>
+<attribute name="TP_SIGNAL_NAME" x="72.39" y="168.91" size="1.778" layer="97"/>
+</instance>
+<instance part="TP8" gate="G$1" x="73.66" y="170.18" smashed="yes">
+<attribute name="NAME" x="72.39" y="171.45" size="1.778" layer="95"/>
+<attribute name="TP_SIGNAL_NAME" x="74.93" y="168.91" size="1.778" layer="97"/>
+</instance>
 </instances>
 <busses>
 <bus name="DPMP1:IC1_RPB10/PWM3H/PMPD0/RB10,IC1_RPB11/PWM9H/PWM3L/PMPD1/RB11,IC1_RPB12/PWM2H/PMPD2/RB12,IC1_RPB13/PWM8H/PWM2L/CTPLS/PMPD3/RB13,IC1_RPB14/PWM1H/VBUSON1/PMPD6/RB14,IC1_RPB15/PWM7H/PWM1L/PMPD7/RB15,IC1_TCK/RPA7/PWM10H/PWM4L/PMPD5/RA7,IC1_TDO/PWM4H/PMPD4/RA10">
 <segment>
-<wire x1="50.8" y1="482.6" x2="73.66" y2="482.6" width="0.762" layer="92"/>
+<wire x1="-12.7" y1="485.14" x2="17.78" y2="485.14" width="0.762" layer="92"/>
 </segment>
 </bus>
@@
 <junction x="12.7" y="40.64"/>
 </segment>
-<segment>
-<wire x1="53.34" y1="482.6" x2="-38.1" y2="396.24" width="0.1524" layer="91"/>
-<wire x1="-38.1" y1="396.24" x2="-38.1" y2="337.82" width="0.1524" layer="91"/>
-<label x="-38.1" y="340.36" size="1.778" layer="95" rot="R90"/>
-<pinref part="IC3" gate="G$1" pin="TCK/RPA7/PWM10H/PWM4L/PMPD5/RA7"/>
-<wire x1="10.16" y1="337.82" x2="-38.1" y2="337.82" width="0.1524" layer="91"/>
-<junction x="10.16" y="337.82"/>
-</segment>
 </net>
 <net name="IC1_RPB14/PWM1H/VBUSON1/PMPD6/RB14" class="0">
@@
 <junction x="12.7" y="38.1"/>
 </segment>
-<segment>
-<wire x1="50.8" y1="482.6" x2="-45.72" y2="391.16" width="0.1524" layer="91"/>
-<wire x1="-45.72" y1="391.16" x2="-45.72" y2="335.28" width="0.1524" layer="91"/>
-<label x="-45.72" y="337.82" size="1.778" layer="95" rot="R90"/>
-<pinref part="IC3" gate="G$1" pin="RPB14/PWM1H/VBUSON1/PMPD6/RB14"/>
-<wire x1="10.16" y1="335.28" x2="-45.72" y2="335.28" width="0.1524" layer="91"/>
-<junction x="10.16" y="335.28"/>
-</segment>
 </net>
 <net name="IC1_RPB15/PWM7H/PWM1L/PMPD7/RB15" class="0">
@@
 <junction x="12.7" y="35.56"/>
 </segment>
-<segment>
-<wire x1="50.8" y1="482.6" x2="-50.8" y2="388.62" width="0.1524" layer="91"/>
-<wire x1="-50.8" y1="388.62" x2="-50.8" y2="332.74" width="0.1524" layer="91"/>
-<label x="-50.8" y="335.28" size="1.778" layer="95" rot="R90"/>
-<pinref part="IC3" gate="G$1" pin="RPB15/PWM7H/PWM1L/PMPD7/RB15"/>
-<wire x1="10.16" y1="332.74" x2="-50.8" y2="332.74" width="0.1524" layer="91"/>
-<junction x="10.16" y="332.74"/>
-</segment>
 </net>
 <net name="IC1_TDO/PWM4H/PMPD4/RA10" class="0">
@@
 <label x="55.88" y="162.56" size="1.778" layer="95" rot="R90" align="bottom-right"/>
 <junction x="55.88" y="104.14"/>
-</segment>
-<segment>
-<wire x1="53.34" y1="482.6" x2="53.34" y2="401.32" width="0.1524" layer="91"/>
+<junction x="55.88" y="167.64"/>
+<pinref part="TP4" gate="G$1" pin="TP"/>
+</segment>
+<segment>
+<wire x1="0" y1="485.14" x2="53.34" y2="444.5" width="0.1524" layer="91"/>
+<wire x1="53.34" y1="444.5" x2="53.34" y2="401.32" width="0.1524" layer="91"/>
 <label x="53.34" y="403.86" size="1.778" layer="95" rot="R90"/>
 <pinref part="IC3" gate="G$1" pin="TDO/PWM4H/PMPD4/RA10"/>
@@
 <label x="58.42" y="165.1" size="1.778" layer="95" rot="R90" align="bottom-right"/>
 <junction x="58.42" y="104.14"/>
-</segment>
-<segment>
-<wire x1="55.88" y1="482.6" x2="55.88" y2="401.32" width="0.1524" layer="91"/>
+<junction x="58.42" y="167.64"/>
+<pinref part="TP5" gate="G$1" pin="TP"/>
+</segment>
+<segment>
+<wire x1="12.7" y1="485.14" x2="55.88" y2="464.82" width="0.1524" layer="91"/>
+<wire x1="55.88" y1="464.82" x2="55.88" y2="401.32" width="0.1524" layer="91"/>
 <label x="55.88" y="403.86" size="1.778" layer="95" rot="R90"/>
 <pinref part="IC3" gate="G$1" pin="RPB13/PWM8H/PWM2L/CTPLS/PMPD3/RB13"/>
@@
 <label x="60.96" y="165.1" size="1.778" layer="95" rot="R90" align="bottom-right"/>
 <junction x="60.96" y="104.14"/>
-</segment>
-<segment>
-<wire x1="58.42" y1="482.6" x2="58.42" y2="447.04" width="0.1524" layer="91"/>
-<wire x1="58.42" y1="447.04" x2="58.42" y2="401.32" width="0.1524" layer="91"/>
-<label x="58.42" y="403.86" size="1.778" layer="95" rot="R90"/>
+<junction x="60.96" y="167.64"/>
+<pinref part="TP6" gate="G$1" pin="TP"/>
+</segment>
+<segment>
+<wire x1="15.24" y1="485.14" x2="58.42" y2="477.52" width="0.1524" layer="91"/>
+<wire x1="58.42" y1="477.52" x2="58.42" y2="401.32" width="0.1524" layer="91"/>
+<label x="58.42" y="434.34" size="1.778" layer="95" rot="R90"/>
 <pinref part="IC3" gate="G$1" pin="RPB12/PWM2H/PMPD2/RB12"/>
 <junction x="58.42" y="401.32"/>
@@
 <label x="71.12" y="165.1" size="1.778" layer="95" rot="R90" align="bottom-right"/>
 <junction x="71.12" y="104.14"/>
-</segment>
-<segment>
-<wire x1="71.12" y1="482.6" x2="68.58" y2="454.66" width="0.1524" layer="91"/>
-<wire x1="68.58" y1="454.66" x2="68.58" y2="401.32" width="0.1524" layer="91"/>
-<label x="68.58" y="403.86" size="1.778" layer="95" rot="R90"/>
+<junction x="71.12" y="167.64"/>
+<pinref part="TP7" gate="G$1" pin="TP"/>
+</segment>
+<segment>
+<wire x1="15.24" y1="485.14" x2="68.58" y2="480.06" width="0.1524" layer="91"/>
+<wire x1="68.58" y1="480.06" x2="68.58" y2="401.32" width="0.1524" layer="91"/>
+<label x="68.58" y="429.26" size="1.778" layer="95" rot="R90"/>
 <pinref part="IC3" gate="G$1" pin="RPB11/PWM9H/PWM3L/PMPD1/RB11"/>
 <junction x="68.58" y="401.32"/>
@@
 <label x="73.66" y="165.1" size="1.778" layer="95" rot="R90" align="bottom-right"/>
 <junction x="73.66" y="104.14"/>
-</segment>
-<segment>
-<wire x1="73.66" y1="482.6" x2="71.12" y2="447.04" width="0.1524" layer="91"/>
-<wire x1="71.12" y1="447.04" x2="71.12" y2="401.32" width="0.1524" layer="91"/>
-<label x="71.12" y="403.86" size="1.778" layer="95" rot="R90"/>
+<junction x="73.66" y="167.64"/>
+<pinref part="TP8" gate="G$1" pin="TP"/>
+</segment>
+<segment>
+<wire x1="15.24" y1="485.14" x2="71.12" y2="482.6" width="0.1524" layer="91"/>
+<wire x1="71.12" y1="482.6" x2="71.12" y2="401.32" width="0.1524" layer="91"/>
+<label x="71.12" y="439.42" size="1.778" layer="95" rot="R90"/>
 <pinref part="IC3" gate="G$1" pin="RPB10/PWM3H/PMPD0/RB10"/>
 <junction x="71.12" y="401.32"/>

Commit message: up
Parts:
- removed TP5, TP6, TP7, TP8: TPB1,27, testpad:TPB1,27
- added TP1, TP2, TP3: TPB1,27, testpad:TPB1,27
Connections:
- removed net IC1_RPB14/PWM1H/VBUSON1/PMPD6/RB14: IC1.RPB14/PWM1H/VBUSON1/PMPD6/RB14
- removed net IC1_RPB15/PWM7H/PWM1L/PMPD7/RB15: IC1.RPB15/PWM7H/PWM1L/PMPD7/RB15
- removed net IC1_TCK/RPA7/PWM10H/PWM4L/PMPD5/RA7: IC1.TCK/RPA7/PWM10H/PWM4L/PMPD5/RA7
- new net N$10: IC1.TCK/RPA7/PWM10H/PWM4L/PMPD5/RA7, IC3.TCK/RPA7/PWM10H/PWM4L/PMPD5/RA7
- new net N$15: IC1.RPB14/PWM1H/VBUSON1/PMPD6/RB14, IC3.RPB14/PWM1H/VBUSON1/PMPD6/RB14
- new net N$17: IC1.RPB15/PWM7H/PWM1L/PMPD7/RB15, IC3.RPB15/PWM7H/PWM1L/PMPD7/RB15
- net IC1_RPB10/PWM3H/PMPD0/RB10: no longer TP8.TP
- net IC1_RPB11/PWM9H/PWM3L/PMPD1/RB11: no longer TP7.TP
- net IC1_RPB12/PWM2H/PMPD2/RB12: no longer TP6.TP
- net IC1_RPB13/PWM8H/PWM2L/CTPLS/PMPD3/RB13: no longer TP5.TP
- net IC1_TDO/PWM4H/PMPD4/RA10: no longer TP4.TP
- net VDD: now also IC1.VDD_5, IC3.VDD_5, TP1.TP, TP2.TP
- net VSS: now also TP3.TP, TP4.TP
Other:
- moved on the sheet: TP4
