File: pic32mk.sch (EAGLE design)
At the start: 39 parts, among them IC1 PIC32MK1024MCF100-I_PT, IC2 ADM3095EBRZ, IC3 PIC32MK1024MCF100-I_PT, IC4 MAX203ECWP

Commit message: up
Parts:
- added TP5, TP6, TP7: TPB1,27, testpad:TPB1,27
Connections:
- net VDD: now also TP5.TP, TP6.TP, TP7.TP
Changed lines of the file:
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@@
 <part name="TP3" library="testpad" library_urn="urn:adsk.eagle:library:385" deviceset="TP" device="B1,27" package3d_urn="urn:adsk.eagle:package:27944/2"/>
 <part name="TP4" library="testpad" library_urn="urn:adsk.eagle:library:385" deviceset="TP" device="B1,27" package3d_urn="urn:adsk.eagle:package:27944/2"/>
+<part name="VDD25" library="supply1" library_urn="urn:adsk.eagle:library:371" deviceset="VDD" device=""/>
+<part name="TP5" library="testpad" library_urn="urn:adsk.eagle:library:385" deviceset="TP" device="B1,27" package3d_urn="urn:adsk.eagle:package:27944/2"/>
+<part name="TP6" library="testpad" library_urn="urn:adsk.eagle:library:385" deviceset="TP" device="B1,27" package3d_urn="urn:adsk.eagle:package:27944/2"/>
+<part name="TP7" library="testpad" library_urn="urn:adsk.eagle:library:385" deviceset="TP" device="B1,27" package3d_urn="urn:adsk.eagle:package:27944/2"/>
 </parts>
 <sheets>
@@
 <attribute name="NAME" x="97.79" y="113.03" size="1.778" layer="95" rot="R270"/>
 <attribute name="TP_SIGNAL_NAME" x="95.25" y="110.49" size="1.778" layer="97" rot="R270"/>
+</instance>
+<instance part="VDD25" gate="G$1" x="88.9" y="426.72" smashed="yes">
+<attribute name="VALUE" x="86.36" y="424.18" size="1.778" layer="96" rot="R90"/>
+</instance>
+<instance part="TP5" gate="G$1" x="86.36" y="424.18" smashed="yes" rot="R90">
+<attribute name="NAME" x="85.09" y="422.91" size="1.778" layer="95" rot="R90"/>
+<attribute name="TP_SIGNAL_NAME" x="87.63" y="425.45" size="1.778" layer="97" rot="R90"/>
+</instance>
+<instance part="TP6" gate="G$1" x="86.36" y="193.04" smashed="yes" rot="R180">
+<attribute name="NAME" x="87.63" y="191.77" size="1.778" layer="95" rot="R180"/>
+<attribute name="TP_SIGNAL_NAME" x="85.09" y="194.31" size="1.778" layer="97" rot="R180"/>
+</instance>
+<instance part="TP7" gate="G$1" x="96.52" y="193.04" smashed="yes" rot="R180">
+<attribute name="NAME" x="97.79" y="191.77" size="1.778" layer="95" rot="R180"/>
+<attribute name="TP_SIGNAL_NAME" x="95.25" y="194.31" size="1.778" layer="97" rot="R180"/>
 </instance>
 </instances>
@@
 <wire x1="10.16" y1="304.8" x2="-7.62" y2="304.8" width="0.1524" layer="91"/>
 <pinref part="VDD19" gate="G$1" pin="VDD"/>
+<junction x="-7.62" y="304.8"/>
 </segment>
 <segment>
@@
 <pinref part="VDD8" gate="G$1" pin="VDD"/>
 <junction x="10.16" y="340.36"/>
+<junction x="-7.62" y="340.36"/>
 </segment>
 <segment>
@@
 <pinref part="VDD9" gate="G$1" pin="VDD"/>
 <junction x="88.9" y="401.32"/>
-<junction x="88.9" y="414.02"/>
 <pinref part="TP2" gate="G$1" pin="TP"/>
 <wire x1="88.9" y1="408.94" x2="88.9" y2="414.02" width="0.1524" layer="91"/>
 <junction x="88.9" y="408.94"/>
+<pinref part="VDD25" gate="G$1" pin="VDD"/>
+<pinref part="TP5" gate="G$1" pin="TP"/>
+<wire x1="88.9" y1="414.02" x2="88.9" y2="424.18" width="0.1524" layer="91"/>
+<junction x="88.9" y="424.18"/>
+<junction x="88.9" y="414.02"/>
 </segment>
 <segment>
 <pinref part="IC3" gate="G$1" pin="VDD_3"/>
 <junction x="81.28" y="208.28"/>
-<wire x1="81.28" y1="208.28" x2="81.28" y2="193.04" width="0.1524" layer="91"/>
+<wire x1="81.28" y1="208.28" x2="81.28" y2="195.58" width="0.1524" layer="91"/>
 <pinref part="VDD20" gate="G$1" pin="VDD"/>
+<wire x1="81.28" y1="195.58" x2="81.28" y2="193.04" width="0.1524" layer="91"/>
+<wire x1="81.28" y1="195.58" x2="86.36" y2="195.58" width="0.1524" layer="91"/>
+<junction x="81.28" y="195.58"/>
+<pinref part="TP6" gate="G$1" pin="TP"/>
+<junction x="86.36" y="195.58"/>
 </segment>
 <segment>
 <pinref part="IC3" gate="G$1" pin="VDD_4"/>
-<wire x1="104.14" y1="193.04" x2="104.14" y2="208.28" width="0.1524" layer="91"/>
+<wire x1="104.14" y1="193.04" x2="104.14" y2="195.58" width="0.1524" layer="91"/>
 <pinref part="VDD10" gate="G$1" pin="VDD"/>
 <junction x="104.14" y="208.28"/>
+<wire x1="104.14" y1="195.58" x2="104.14" y2="208.28" width="0.1524" layer="91"/>
+<wire x1="96.52" y1="195.58" x2="104.14" y2="195.58" width="0.1524" layer="91"/>
+<junction x="104.14" y="195.58"/>
+<pinref part="TP7" gate="G$1" pin="TP"/>
+<junction x="96.52" y="195.58"/>
 </segment>
 <segment>
@@
 <pinref part="IC3" gate="G$1" pin="!MCLR"/>
 <pinref part="R3" gate="G$1" pin="2"/>
-<wire x1="10.16" y1="312.42" x2="-27.94" y2="312.42" width="0.1524" layer="91"/>
 <junction x="10.16" y="312.42"/>
 <pinref part="SV1" gate="1" pin="1"/>
+<wire x1="10.16" y1="312.42" x2="-30.48" y2="312.42" width="0.1524" layer="91"/>
 <wire x1="-30.48" y1="312.42" x2="-33.02" y2="312.42" width="0.1524" layer="91"/>
 <wire x1="-55.88" y1="193.04" x2="-30.48" y2="193.04" width="0.1524" layer="91"/>
 <wire x1="-30.48" y1="193.04" x2="-30.48" y2="226.06" width="0.1524" layer="91"/>
 <wire x1="-30.48" y1="226.06" x2="-30.48" y2="312.42" width="0.1524" layer="91"/>
-<wire x1="-30.48" y1="312.42" x2="-27.94" y2="312.42" width="0.1524" layer="91"/>
 <junction x="-33.02" y="312.42"/>
 <junction x="-30.48" y="312.42"/>

Commit message: up
Parts:
- removed C5, C8, C9: 0.1, rcl:C-USC0805
- removed L2: 1000, inductor-neosid:SM-1206
- removed R3: 1k, rcl:R-US_M0805
- removed R4: 10k, rcl:R-US_M0805
- removed S2: B3W-9000-Y1N, B3W-9000-Y1N:B3W-9000-Y1N
- removed SV1: ICSP1, con-lstb:MA06-1
- removed TP2, TP3, TP5, TP6, TP7: TPB1,27, testpad:TPB1,27
- added IC5: MC33931EK, MC33931EK:MC33931EK
- IC3: value PIC32MK1024MCF100-I_PT -> MC33931EK; device PIC32MK1024MCF100-I_PT:PIC32MK1024MCF100-I_PT -> MC33931EK:MC33931EK
Connections:
- removed net IC1_RPB10/PWM3H/PMPD0/RB10: IC1.RPB10/PWM3H/PMPD0/RB10, IC3.RPB10/PWM3H/PMPD0/RB10
- removed net IC1_RPB11/PWM9H/PWM3L/PMPD1/RB11: IC1.RPB11/PWM9H/PWM3L/PMPD1/RB11, IC3.RPB11/PWM9H/PWM3L/PMPD1/RB11
- removed net IC1_RPB12/PWM2H/PMPD2/RB12: IC1.RPB12/PWM2H/PMPD2/RB12, IC3.RPB12/PWM2H/PMPD2/RB12
- removed net IC1_RPB13/PWM8H/PWM2L/CTPLS/PMPD3/RB13: IC1.RPB13/PWM8H/PWM2L/CTPLS/PMPD3/RB13, IC3.RPB13/PWM8H/PWM2L/CTPLS/PMPD3/RB13
- removed net IC1_TDO/PWM4H/PMPD4/RA10: IC1.TDO/PWM4H/PMPD4/RA10, IC3.TDO/PWM4H/PMPD4/RA10
- removed net N$10: IC1.TCK/RPA7/PWM10H/PWM4L/PMPD5/RA7, IC3.TCK/RPA7/PWM10H/PWM4L/PMPD5/RA7
- removed net N$11: IC3.PGED1/OA1IN-/AN5/CTCMP/C1IN1-/RTCC/RPB3/RB3, SV1.4
- removed net N$12: IC3.PGEC1/OA1IN+/AN4/C1IN1+/C1IN3-/C2IN3-/RPB2/RB2, SV1.5
- removed net N$15: IC1.RPB14/PWM1H/VBUSON1/PMPD6/RB14, IC3.RPB14/PWM1H/VBUSON1/PMPD6/RB14
- removed net N$17: IC1.RPB15/PWM7H/PWM1L/PMPD7/RB15, IC3.RPB15/PWM7H/PWM1L/PMPD7/RB15
- removed net N$4: C5.1, R3.1, R4.1, S2.4
- removed net N$5: IC3.!MCLR, R3.2, SV1.1
- removed net N$8: C8.1, IC3.AVDD, L2.2
- net +3V3: no longer SV1.3
- net N$16: no longer IC3.SOSCO/RPB8(4)/RB8(4)
- net N$7: no longer IC3.OSCI/CLKI/AN49/CVD49/RPC12/RC12
- net VDD: no longer C9.1, IC3.VDD_1, IC3.VDD_2, IC3.VDD_3, IC3.VDD_4, IC3.VDD_5, IC3.VDD_6, IC3.VUSB3V3, L2.1, R4.2, TP2.TP, TP5.TP, TP6.TP, TP7.TP
- net VSS: no longer C5.2, C8.2, C9.2, IC3.AVSS, IC3.VSS_1, IC3.VSS_2, IC3.VSS_3, IC3.VSS_4, IC3.VSS_5, IC3.VSS_6, S2.2, SV1.2, TP3.TP
Other:
- moved on the sheet: C10, C11, F1, F2, R5, R6, S3, U$2
